File: hardware/mp3triggerv3.sch (EAGLE design)
At the start: 0 parts

Commit message: added Jamie's project files
Parts:
- added C1: 10uF, SparkFun-Capacitors:CAP1206
- added C10, C13, C15, C18, C19, C21, C22, C23, C24, C25, C26, C4, C9: 0.1uF, SparkFun-Capacitors:CAP0603-CAP
- added C11, C30, C31: 1uF, SparkFun-Capacitors:CAP0603-CAP
- added C12: 4.7uF, SparkFun-Capacitors:CAP0603-CAP
- added C14, C20: 2.2uF, SparkFun-Capacitors:CAP0603-CAP
- added C16, C17: 33pF, SparkFun-Capacitors:CAP0402-CAP
- added C2: 10uF, SparkFun-Capacitors:1UF-25V-10%(0805)
- added C27: 10uF, SparkFun-Capacitors:CAP0603-CAP
- added C28, C29: 2200pF, SparkFun-Capacitors:CAP0603-CAP
- added C3, C5: 2.2uF, SparkFun-Capacitors:1UF-25V-10%(0805)
- added J1: 5.5x2.1mm Barrel, SparkFun-Connectors:POWER_JACKSMD
- added J2: (no value), SparkFun-Connectors:AUDIO-JACKSMD2
- added J3: USD-SOCKETNEW, robertsonics:USD-SOCKETNEW
- added J4: (no value), SparkFun-Connectors:M06SIP
- added J5, JP2, JP3: (no value), SparkFun-Connectors:M02PTH
- added J6: M08X2, SparkFun-Connectors:M08X2
- added J7: (no value), SparkFun-Connectors:M04PTH
- added J8: M10X2, SparkFun-Connectors:M10X2
- added JP1: (no value), SparkFun-Connectors:M03PTH
- added LED1: (no value), SparkFun-LED:LED0603
- added R1, R2, R3, R4, R5: 47K, SparkFun-Passives:RESISTOR0603-RES
- added R10, R9: 22K, SparkFun-Passives:RESISTOR0603-RES
- added R11, R12, R13, R14, R15, R16, R17, R18, R20, R29, R30, R31, R32, R33, R34, R35, R36, R8: 10K, SparkFun-Passives:RESISTOR0603-RES
- added R19: 330, SparkFun-Passives:RESISTOR0603-RES
- added R21, R22, R23, R24, R25, R26, R27, R28: 100, SparkFun-Passives:RESISTOR0603-RES
- added R6, R7: 470, SparkFun-Passives:RESISTOR0603-RES
- added S1: NAV_SWITCHSMD, SparkFun-Electromechanical:NAV_SWITCHSMD
- added U1: NCP1117, SparkFun-PowerIC:V_REG_LM1117SOT223
- added U2: MIC5323-3.3, SparkFun-PowerIC:MIC52053.3V
- added U4: STM32F405RG, robertsonics:STM32F405RG
- added U5: PCM5100, robertsonics:PCM5100
- added U6: LM4990, robertsonics:LM4990
- added Y1: 8MHz, SparkFun-FreqCtrl:CRYSTALSMD
Connections:
- new net +5V: C2.1, C3.1, C31.2, J7.4, JP2.2, U1.OUT, U1.OUT@1, U2.EN, U2.IN, U6.VDD
- new net AMPENA: R8.2, U4.PC3, U6.SHTDN
- new net AMPIN: JP3.2, R9.1
- new net BOOT0: JP1.2, U4.BOOT0
- new net DEMP: U4.PC2, U5.DEMP
- new net FILTER: U4.PC1, U5.FLT
- new net GND: C1.2, C10.2, C11.2, C12.2, C13.2, C14.2, C15.2, C16.1, C17.1, C18.2, C19.2, C2.2, C20.2, C21.1, C22.2, C23.1, C25.2, C26.1, C27.1, C28.1, C29.1, C3.2, C30.1, C31.1, C4.2, C5.2, J1.GND, J1.GNDBREAK, J2.SLEEVE, J3.GND, J3.SHIELD@1, J3.SHIELD@3, J3.SHIELD@4, J4.1, J6.1, J6.11, J6.13, J6.15, J6.3, J6.5, J6.7, J6.9, J7.1, J8.10, J8.12, J8.14, J8.16, J8.18, J8.20, J8.4, J8.6, J8.8, R11.1, R12.1, R13.1, R16.2, R20.2, R8.1, S1.C, U1.ADJ, U2.GND, U4.VSS1, U4.VSS2, U4.VSSA, U5.AGND, U5.CPGND, U5.DGND, U5.FMT, U6.GND
- new net I2S_BCLK: U4.PB13/I2S2_CK, U5.BCK
- new net I2S_DOUT: U4.PB15/I2S2_SD, U5.DIN
- new net I2S_LRCK: U4.PB12/I2S2_WS, U5.LRCK
- new net I2S_MCLK: U4.PC6/I2S2_MCK, U5.SCK
- new net JTCK: J8.9, U4.PA14/JTCK
- new net JTDI: J8.5, U4.PA15/JTDI
- new net JTDO: J8.13, U4.PB3/JTDO
- new net JTMS: J8.7, U4.PA13/JTMS
- new net JTRST: J8.3, U4.PB4/JTRST
- new net LED1: LED1.C, U4.PC4
- new net LOUTL: C28.2, J2.LEFT, JP3.1, R7.2
- new net LOUTR: C29.2, J2.RIGHT, R6.2
- new net MUTE: U4.PC0, U5.XSMT
- new net N$10: JP1.3, R17.2
- new net N$11: LED1.A, R19.2
- new net N$12: R20.1, U4.PB2-BOOT1
- new net N$13: J8.19, R11.2
- new net N$14: C23.2, U5.LDOO
- new net N$15: R6.1, U5.OUTR
- new net N$16: C24.2, U5.CAPP
- new net N$17: C24.1, U5.CAPM
- new net N$18: C25.1, U5.VNEG
- new net N$19: R7.1, U5.OUTL
- new net N$2: C4.1, U2.BP
- new net N$20: C30.2, U6.+IN, U6.BYPASS
- new net N$21: J8.17, R12.2
- new net N$22: J8.11, R13.2
- new net N$23: J6.2, R21.1, R36.1
- new net N$24: J6.4, R22.1, R35.1
- new net N$25: J6.6, R23.1, R34.1
- new net N$26: J6.8, R24.1, R33.1
- new net N$27: J6.10, R25.1, R32.1
- new net N$28: J6.12, R26.1, R31.1
- new net N$29: R10.1, R9.2, U6.-IN
- new net N$3: C9.2, U4.VBAT
- new net N$30: J6.14, R27.1, R30.1
- new net N$31: J6.16, R28.1, R29.1
- new net N$32: J4.3, JP2.1
- new net N$4: C14.1, U4.VCAP1
- new net N$5: C16.2, U4.PH0, Y1.2
- new net N$6: C17.2, U4.PH1, Y1.1
- new net N$7: JP1.1, R16.1
- new net N$8: C20.1, U4.VCAP2
- new net N$9: J4.4, R15.2
- new net NAV1: S1.1, U4.PC13
- new net NAV2: S1.2, U4.PC15
- new net NAVT: S1.T, U4.PC14
- new net NRST: J8.15, R18.1, U4.NRST
- new net PLAYOUT: J7.2, U4.PC5
- new net RXD: R14.1, R15.1, U4.PA10/UART1_RX
- new net SD_CD: J3.SHIELD@2, U4.PB0
- new net SD_CK: J3.SCK, U4.PC12/SDIO_CLK
- new net SD_CMD: J3.DI, R3.1, U4.PD2/SDIO_CMD
- new net SD_D0: J3.DO, R2.1, U4.PC8/SDIO_D0
- new net SD_D1: J3.RSV, R1.1, U4.PC9/SDIO_D1
- new net SD_D2: J3.NC, R5.1, U4.PC10/SDIO_D2
- new net SD_D3: J3.CS, R4.1, U4.PC11/SDIO_D3
- new net SPKR+: J5.2, U6.VO2
- new net SPKR-: J5.1, R10.2, U6.VO1
- new net TRIG00: R21.2, U4.PA0
- new net TRIG01: R22.2, U4.PA1
- new net TRIG02: R23.2, U4.PA2/UART2_TX
- new net TRIG03: R24.2, U4.PA3/UART2_RX
- new net TRIG04: R25.2, U4.PA4/SPI1_NSS
- new net TRIG05: R26.2, U4.PA5/SPI1_SCK
- new net TRIG06: R27.2, U4.PA6/SPI1_MISO
- new net TRIG07: R28.2, U4.PA7/SPI1_MOSI
- new net TXD: J4.5, U4.PA9/UART1_TX
- new net VCC: C10.1, C11.1, C12.1, C13.1, C15.1, C18.1, C19.1, C21.2, C22.1, C26.2, C27.2, C5.1, C9.1, J3.VCC, J7.3, J8.1, J8.2, R1.2, R14.2, R17.1, R18.2, R19.1, R2.2, R29.2, R3.2, R30.2, R31.2, R32.2, R33.2, R34.2, R35.2, R36.2, R4.2, R5.2, U2.OUT, U4.VDD1, U4.VDD2, U4.VDD3, U4.VDD4, U4.VDDA, U5.AVDD, U5.CPVDD, U5.DVDD
- new net VIN_9V: C1.1, J1.PWR, U1.IN
