File: hardware/mp3triggerv3.sch (EAGLE design)
At the start: 83 parts, among them J1 5.5x2.1mm Barrel, J3 USD-SOCKETNEW, J6 M08X2, J8 M10X2, U1 NCP1117, U2 MIC5323-3.3, U4 STM32F405RG, U5 PCM5100, U6 LM4990, Y1 8MHz

Commit message: v010
files sent to Jamie
Parts:
- removed J6: M08X2, SparkFun-Connectors:M08X2
- removed J7: (no value), SparkFun-Connectors:M04PTH
- removed J8: M10X2, SparkFun-Connectors:M10X2
- removed R11, R12, R13, R18, R29, R30, R31, R32, R33, R34, R35, R36: 10K, SparkFun-Passives:RESISTOR0603-RES
- removed R21, R22, R23, R24, R25, R26, R27, R28: 100, SparkFun-Passives:RESISTOR0603-RES
- added C6: 3.3V jumper, SparkFun-Capacitors:1UF-25V-10%(0805)
- added C7: GND jumper, SparkFun-Capacitors:1UF-25V-10%(0805)
- added C8: 5V jumper, SparkFun-Capacitors:1UF-25V-10%(0805)
- added J10: M08X2, SparkFun-Connectors:M08X2
- added J11: (no value), SparkFun-Connectors:M04PTH
- added J9: M10X2, SparkFun-Connectors:M10X2
- added JP4, JP5, JP6: M01PTH, SparkFun-Connectors:M01PTH
- added R37, R38, R39, R40, R49, R50, R51, R52, R53, R54, R55, R56: 10K, SparkFun-Passives:RESISTOR0603-RES
- added R41, R42, R43, R44, R45, R46, R47, R48: 100, SparkFun-Passives:RESISTOR0603-RES
- added STANDOFF1, STANDOFF2, STANDOFF3, STANDOFF4: STAND-OFF, SparkFun-Electromechanical:STAND-OFF
Connections:
- removed net N$13: J8.19, R11.2
- removed net N$21: J8.17, R12.2
- removed net N$22: J8.11, R13.2
- removed net N$23: J6.2, R21.1, R36.1
- removed net N$24: J6.4, R22.1, R35.1
- removed net N$25: J6.6, R23.1, R34.1
- removed net N$26: J6.8, R24.1, R33.1
- removed net N$27: J6.10, R25.1, R32.1
- removed net N$28: J6.12, R26.1, R31.1
- removed net N$30: J6.14, R27.1, R30.1
- removed net N$31: J6.16, R28.1, R29.1
- new net N$1: J9.19, R37.2
- new net N$33: J9.17, R38.2
- new net N$34: J9.11, R39.2
- new net N$35: J10.2, R41.1, R56.1
- new net N$36: J10.4, R42.1, R55.1
- new net N$37: J10.6, R43.1, R54.1
- new net N$38: J10.8, R44.1, R53.1
- new net N$39: J10.10, R45.1, R52.1
- new net N$40: J10.12, R46.1, R51.1
- new net N$41: J10.14, R47.1, R50.1
- new net N$42: J10.16, R48.1, R49.1
- net +5V: now also C8.1, C8.2, J11.4, JP4.1; no longer J7.4
- net GND: now also C7.1, C7.2, J10.1, J10.11, J10.13, J10.15, J10.3, J10.5, J10.7, J10.9, J11.1, J9.10, J9.12, J9.14, J9.16, J9.18, J9.20, J9.4, J9.6, J9.8, JP6.1, R37.1, R38.1, R39.1; no longer J6.1, J6.11, J6.13, J6.15, J6.3, J6.5, J6.7, J6.9, J7.1, J8.10, J8.12, J8.14, J8.16, J8.18, J8.20, J8.4, J8.6, J8.8, R11.1, R12.1, R13.1
- net JTCK: now also J9.9; no longer J8.9
- net JTDI: now also J9.5; no longer J8.5
- net JTDO: now also J9.13; no longer J8.13
- net JTMS: now also J9.7; no longer J8.7
- net JTRST: now also J9.3; no longer J8.3
- net NRST: now also J9.15, R40.1; no longer J8.15, R18.1
- net PLAYOUT: now also J11.2; no longer J7.2
- net TRIG00: now also R41.2; no longer R21.2
- net TRIG01: now also R42.2; no longer R22.2
- net TRIG02: now also R43.2; no longer R23.2
- net TRIG03: now also R44.2; no longer R24.2
- net TRIG04: now also R45.2; no longer R25.2
- net TRIG05: now also R46.2; no longer R26.2
- net TRIG06: now also R47.2; no longer R27.2
- net TRIG07: now also R48.2; no longer R28.2
- net VCC: now also C6.1, C6.2, J11.3, J9.1, J9.2, JP5.1, R40.2, R49.2, R50.2, R51.2, R52.2, R53.2, R54.2, R55.2, R56.2; no longer J7.3, J8.1, J8.2, R18.2, R29.2, R30.2, R31.2, R32.2, R33.2, R34.2, R35.2, R36.2

Commit message: v31, ready for review
Parts:
- removed J10: M08X2, SparkFun-Connectors:M08X2
- removed J11: (no value), SparkFun-Connectors:M04PTH
- removed J9: M10X2, SparkFun-Connectors:M10X2
- removed JP2, JP3: (no value), SparkFun-Connectors:M02PTH
- removed JP4, JP5, JP6: M01PTH, SparkFun-Connectors:M01PTH
- removed R49, R50, R51, R52, R53, R54, R55, R56: 10K, SparkFun-Passives:RESISTOR0603-RES
- removed S1: NAV_SWITCHSMD, SparkFun-Electromechanical:NAV_SWITCHSMD
- added CC_TEXT1: CREATIVE_COMMONS, SparkFun-Aesthetics:CREATIVE_COMMONS
- added J6, J7: M08X2, SparkFun-Connectors:M08X2
- added J8: (no value), SparkFun-Connectors:M04PTH
- added LOGO1: OSHW-LOGOL, SparkFun-Aesthetics:OSHW-LOGOL
- added LOGO2: LOGO-SFENEW, SparkFun-Aesthetics:LOGO-SFENEW
- added LOGO3: LOGO-SFESK, SparkFun-Aesthetics:LOGO-SFESK
- added R11, R12, R13, R18, R21, R22, R23, R24, R33, R34, R35, R36: 100, SparkFun-Passives:RESISTOR0603-RES
- added R25, R26, R27, R28, R29, R30, R31, R32: 10K, SparkFun-Passives:RESISTOR0603-RES
- added SJ1: SOLDERJUMPERTRACE, SparkFun-Passives:SOLDERJUMPERTRACE
- added SJ2: SOLDERJUMPERNO, SparkFun-Passives:SOLDERJUMPERNO
- C16, C17: device SparkFun-Capacitors:CAP0402-CAP -> SparkFun-Capacitors:CAP0603-CAP
- R10: value 22K -> 10K
- R15, R37, R38, R39, R40: value 10K -> 100
- R41, R42, R43, R44, R45, R46, R47, R48: value 100 -> 10K
Connections:
- removed net JTCK: J9.9, U4.PA14/JTCK
- removed net JTDI: J9.5, U4.PA15/JTDI
- removed net JTDO: J9.13, U4.PB3/JTDO
- removed net JTMS: J9.7, U4.PA13/JTMS
- removed net JTRST: J9.3, U4.PB4/JTRST
- removed net N$33: J9.17, R38.2
- removed net N$34: J9.11, R39.2
- removed net NAV1: S1.1, U4.PC13
- removed net NAV2: S1.2, U4.PC15
- removed net NAVT: S1.T, U4.PC14
- new net N$23: J6.4, R12.1, R31.1
- new net N$24: J6.6, R13.1, R30.1
- new net N$25: J6.8, R18.1, R29.1
- new net N$26: J6.10, R21.1, R28.1
- new net N$27: J6.12, R22.1, R27.1
- new net N$28: J6.14, R23.1, R26.1
- new net N$30: J6.16, R24.1, R25.1
- new net TRIG08: R11.2, U4.PB8
- new net TRIG09: R12.2, U4.PB9
- new net TRIG10: R13.2, U4.PB10
- new net TRIG11: R18.2, U4.PA11
- new net TRIG12: R21.2, U4.PA12
- new net TRIG13: R22.2, U4.PA13/JTMS
- new net TRIG14: R23.2, U4.PA14/JTCK
- new net TRIG15: R24.2, U4.PA15/JTDI
- net +5V: now also J8.4, SJ2.2; no longer J11.4, JP2.2, JP4.1
- net AMPIN: now also SJ1.2; no longer JP3.2
- net GND: now also J6.1, J6.11, J6.13, J6.15, J6.3, J6.5, J6.7, J6.9, J7.1, J7.11, J7.13, J7.15, J7.3, J7.5, J7.7, J7.9, J8.1; no longer J10.1, J10.11, J10.13, J10.15, J10.3, J10.5, J10.7, J10.9, J11.1, J9.10, J9.12, J9.14, J9.16, J9.18, J9.20, J9.4, J9.6, J9.8, JP6.1, R37.1, R38.1, R39.1, S1.C
- net LOUTL: now also SJ1.1; no longer JP3.1
- net N$1: now also J6.2, R11.1, R32.1; no longer J9.19, R37.2
- net N$32: now also SJ2.1; no longer JP2.1
- net N$35: now also J7.2, R40.1, R48.1; no longer J10.2, R41.1, R56.1
- net N$36: now also J7.4, R39.1, R47.1; no longer J10.4, R42.1, R55.1
- net N$37: now also J7.6, R38.1, R46.1; no longer J10.6, R43.1, R54.1
- net N$38: now also J7.8, R37.1, R45.1; no longer J10.8, R44.1, R53.1
- net N$39: now also J7.10, R36.1, R44.1; no longer J10.10, R45.1, R52.1
- net N$40: now also J7.12, R35.1, R43.1; no longer J10.12, R46.1, R51.1
- net N$41: now also J7.14, R34.1, R42.1; no longer J10.14, R47.1, R50.1
- net N$42: now also J7.16, R33.1, R41.1; no longer J10.16, R48.1, R49.1
- net NRST: no longer J9.15, R40.1
- net PLAYOUT: now also J8.2; no longer J11.2
- net TRIG00: now also R40.2; no longer R41.2
- net TRIG01: now also R39.2; no longer R42.2
- net TRIG02: now also R38.2; no longer R43.2
- net TRIG03: now also R37.2; no longer R44.2
- net TRIG04: now also R36.2; no longer R45.2
- net TRIG05: now also R35.2; no longer R46.2
- net TRIG06: now also R34.2; no longer R47.2
- net TRIG07: now also R33.2; no longer R48.2
- net VCC: now also J8.3, R25.2, R26.2, R27.2, R28.2, R29.2, R30.2, R31.2, R32.2, R41.2, R42.2, R43.2, R44.2, R45.2, R46.2, R47.2, R48.2; no longer J11.3, J9.1, J9.2, JP5.1, R40.2, R49.2, R50.2, R51.2, R52.2, R53.2, R54.2, R55.2, R56.2
Other:
- note added: "Jamie Robertson, Jordan McConnell"
- moved on the sheet: C10, C11, C12, C13, C14, C15, C16, C17, C18, C19, C20, C9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

Commit message: v31, ready for protos, now dubbed 'pro' version
Parts:
- removed C6: 3.3V jumper, SparkFun-Capacitors:1UF-25V-10%(0805)
- removed C7: GND jumper, SparkFun-Capacitors:1UF-25V-10%(0805)
- removed C8: 5V jumper, SparkFun-Capacitors:1UF-25V-10%(0805)
- added SJ3, SJ4, SJ5: SOLDERJUMPERTRACE, SparkFun-Passives:SOLDERJUMPERTRACE
- C1: device SparkFun-Capacitors:CAP1206 -> SparkFun-Capacitors:10UF50V20%(1210)
Connections:
- net +5V: now also SJ3.1, SJ3.2; no longer C8.1, C8.2
- net GND: now also SJ5.1, SJ5.2; no longer C7.1, C7.2
- net VCC: now also SJ4.1, SJ4.2; no longer C6.1, C6.2
Other:
- note added: "3.3V jumper"
- note added: "5V jumper"
- note added: "GND jumper"
Changed lines of the file:
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@@
 <part name="GND5" library="supply1" deviceset="GND" device=""/>
 <part name="P+4" library="supply1" deviceset="VCC" device="" value="+3V3"/>
-<part name="C1" library="SparkFun-Capacitors" deviceset="CAP" device="1206" value="10uF"/>
+<part name="C1" library="SparkFun-Capacitors" deviceset="10UF50V20%(1210)" device="" value="10uF"/>
 <part name="C9" library="SparkFun-Capacitors" deviceset="CAP" device="0603-CAP" value="0.1uF"/>
 <part name="P+5" library="supply1" deviceset="VCC" device="" value="+3V3"/>
@@
 <part name="GND29" library="supply1" deviceset="GND" device=""/>
 <part name="J8" library="SparkFun-Connectors" deviceset="M04" device="PTH"/>
-<part name="C6" library="SparkFun-Capacitors" deviceset="1UF-25V-10%(0805)" device="" value="3.3V jumper"/>
-<part name="C7" library="SparkFun-Capacitors" deviceset="1UF-25V-10%(0805)" device="" value="GND jumper"/>
 <part name="P+12" library="supply1" deviceset="VCC" device="" value="+3V3"/>
 <part name="P+15" library="supply1" deviceset="VCC" device="" value="+3V3"/>
 <part name="GND28" library="supply1" deviceset="GND" device=""/>
 <part name="GND32" library="supply1" deviceset="GND" device=""/>
-<part name="C8" library="SparkFun-Capacitors" deviceset="1UF-25V-10%(0805)" device="" value="5V jumper"/>
 <part name="P+17" library="supply1" deviceset="+5V" device=""/>
 <part name="P+18" library="supply1" deviceset="+5V" device=""/>
@@
 <part name="LOGO2" library="SparkFun-Aesthetics" deviceset="LOGO-SFE" device="NEW"/>
 <part name="LOGO3" library="SparkFun-Aesthetics" deviceset="LOGO-SFE" device="SK"/>
+<part name="SJ3" library="SparkFun-Passives" deviceset="SOLDERJUMPER" device="TRACE"/>
+<part name="SJ4" library="SparkFun-Passives" deviceset="SOLDERJUMPER" device="TRACE"/>
+<part name="SJ5" library="SparkFun-Passives" deviceset="SOLDERJUMPER" device="TRACE"/>
 </parts>
 <sheets>
@@
 <wire x1="76.2" y1="147.32" x2="76.2" y2="137.16" width="0.4064" layer="97" style="shortdash"/>
 <text x="22.86" y="5.08" size="1.778" layer="94">Jamie Robertson, Jordan McConnell</text>
+<text x="10.16" y="139.7" size="1.778" layer="95">5V jumper</text>
+<text x="30.48" y="139.7" size="1.778" layer="95">3.3V jumper</text>
+<text x="55.88" y="139.7" size="1.778" layer="95">GND jumper</text>
 </plain>
 <instances>
@@
 <instance part="GND29" gate="1" x="292.1" y="200.66"/>
 <instance part="J8" gate="G$1" x="129.54" y="172.72"/>
-<instance part="C6" gate="G$1" x="43.18" y="147.32" smashed="yes" rot="R90">
-<attribute name="VALUE" x="50.8" y="144.907" size="1.778" layer="96" rot="R180"/>
-</instance>
-<instance part="C7" gate="G$1" x="63.5" y="147.32" smashed="yes" rot="R90">
-<attribute name="VALUE" x="70.358" y="144.907" size="1.778" layer="96" rot="R180"/>
-</instance>
-<instance part="P+12" gate="VCC" x="50.8" y="152.4"/>
-<instance part="P+15" gate="VCC" x="33.02" y="152.4"/>
-<instance part="GND28" gate="1" x="55.88" y="142.24"/>
-<instance part="GND32" gate="1" x="68.58" y="142.24"/>
-<instance part="C8" gate="G$1" x="20.32" y="147.32" smashed="yes" rot="R90">
-<attribute name="VALUE" x="27.432" y="145.161" size="1.778" layer="96" rot="R180"/>
-</instance>
-<instance part="P+17" gate="1" x="12.7" y="152.4"/>
-<instance part="P+18" gate="1" x="25.4" y="152.4"/>
+<instance part="P+12" gate="VCC" x="45.72" y="149.86"/>
+<instance part="P+15" gate="VCC" x="30.48" y="149.86"/>
+<instance part="GND28" gate="1" x="55.88" y="144.78"/>
+<instance part="GND32" gate="1" x="71.12" y="144.78"/>
+<instance part="P+17" gate="1" x="7.62" y="149.86"/>
+<instance part="P+18" gate="1" x="22.86" y="149.86"/>
 <instance part="SJ1" gate="1" x="106.68" y="20.32"/>
 <instance part="SJ2" gate="1" x="119.38" y="231.14" rot="R90"/>
@@
 <instance part="LOGO2" gate="G$1" x="299.72" y="7.62"/>
 <instance part="LOGO3" gate="G$1" x="299.72" y="15.24"/>
+<instance part="SJ3" gate="1" x="15.24" y="144.78" smashed="yes">
+<attribute name="NAME" x="12.7" y="147.32" size="1.778" layer="95"/>
+</instance>
+<instance part="SJ4" gate="1" x="38.1" y="144.78" smashed="yes">
+<attribute name="NAME" x="35.56" y="147.32" size="1.778" layer="95"/>
+</instance>
+<instance part="SJ5" gate="1" x="63.5" y="149.86" smashed="yes">
+<attribute name="NAME" x="60.96" y="152.4" size="1.778" layer="95"/>
+</instance>
 </instances>
 <busses>
@@
 </segment>
 <segment>
-<pinref part="C7" gate="G$1" pin="1"/>
-<wire x1="58.42" y1="147.32" x2="55.88" y2="147.32" width="0.1524" layer="91"/>
-<wire x1="55.88" y1="147.32" x2="55.88" y2="144.78" width="0.1524" layer="91"/>
+<wire x1="58.42" y1="149.86" x2="55.88" y2="149.86" width="0.1524" layer="91"/>
+<wire x1="55.88" y1="149.86" x2="55.88" y2="147.32" width="0.1524" layer="91"/>
 <pinref part="GND28" gate="1" pin="GND"/>
-</segment>
-<segment>
-<pinref part="C7" gate="G$1" pin="2"/>
-<wire x1="66.04" y1="147.32" x2="68.58" y2="147.32" width="0.1524" layer="91"/>
-<wire x1="68.58" y1="147.32" x2="68.58" y2="144.78" width="0.1524" layer="91"/>
+<pinref part="SJ5" gate="1" pin="1"/>
+</segment>
+<segment>
+<wire x1="68.58" y1="149.86" x2="71.12" y2="149.86" width="0.1524" layer="91"/>
+<wire x1="71.12" y1="149.86" x2="71.12" y2="147.32" width="0.1524" layer="91"/>
 <pinref part="GND32" gate="1" pin="GND"/>
+<pinref part="SJ5" gate="1" pin="2"/>
 </segment>
 <segment>
@@
 </segment>
 <segment>
-<pinref part="C8" gate="G$1" pin="2"/>
 <pinref part="P+18" gate="1" pin="+5V"/>
-<wire x1="22.86" y1="147.32" x2="25.4" y2="147.32" width="0.1524" layer="91"/>
-<wire x1="25.4" y1="147.32" x2="25.4" y2="149.86" width="0.1524" layer="91"/>
-</segment>
-<segment>
-<pinref part="C8" gate="G$1" pin="1"/>
+<wire x1="20.32" y1="144.78" x2="22.86" y2="144.78" width="0.1524" layer="91"/>
+<wire x1="22.86" y1="144.78" x2="22.86" y2="147.32" width="0.1524" layer="91"/>
+<pinref part="SJ3" gate="1" pin="2"/>
+</segment>
+<segment>
 <pinref part="P+17" gate="1" pin="+5V"/>
-<wire x1="15.24" y1="147.32" x2="12.7" y2="147.32" width="0.1524" layer="91"/>
-<wire x1="12.7" y1="147.32" x2="12.7" y2="149.86" width="0.1524" layer="91"/>
+<wire x1="10.16" y1="144.78" x2="7.62" y2="144.78" width="0.1524" layer="91"/>
+<wire x1="7.62" y1="144.78" x2="7.62" y2="147.32" width="0.1524" layer="91"/>
+<pinref part="SJ3" gate="1" pin="1"/>
 </segment>
 <segment>
@@
 </segment>
 <segment>
-<pinref part="C6" gate="G$1" pin="2"/>
-<wire x1="45.72" y1="147.32" x2="50.8" y2="147.32" width="0.1524" layer="91"/>
-<wire x1="50.8" y1="147.32" x2="50.8" y2="149.86" width="0.1524" layer="91"/>
+<wire x1="43.18" y1="144.78" x2="45.72" y2="144.78" width="0.1524" layer="91"/>
+<wire x1="45.72" y1="144.78" x2="45.72" y2="147.32" width="0.1524" layer="91"/>
 <pinref part="P+12" gate="VCC" pin="VCC"/>
-</segment>
-<segment>
-<pinref part="C6" gate="G$1" pin="1"/>
-<wire x1="38.1" y1="147.32" x2="33.02" y2="147.32" width="0.1524" layer="91"/>
-<wire x1="33.02" y1="147.32" x2="33.02" y2="149.86" width="0.1524" layer="91"/>
+<pinref part="SJ4" gate="1" pin="2"/>
+</segment>
+<segment>
+<wire x1="33.02" y1="144.78" x2="30.48" y2="144.78" width="0.1524" layer="91"/>
+<wire x1="30.48" y1="144.78" x2="30.48" y2="147.32" width="0.1524" layer="91"/>
 <pinref part="P+15" gate="VCC" pin="VCC"/>
-</segment>
-<segment>
+<pinref part="SJ4" gate="1" pin="1"/>
+</segment>
+<segment>
