File: hardware/mp3triggerv3.brd (EAGLE design)
At the start: 63.5 x 58.4 mm, 105 parts, among them J1 5.5x2.1mm Barrel, J3 USD-SOCKETNEW, J6 M08X2, J7 M08X2, U1 NCP1117, U2 MIC5323-3.3, U4 STM32F405RG, U5 PCM5100, U6 LM4990, Y1 8MHz

Commit message: v31, ready for protos, now dubbed 'pro' version
Parts:
- removed C6: 3.3V jumper, SparkFun-Capacitors:0805
- removed C7: GND jumper, SparkFun-Capacitors:0805
- removed C8: 5V jumper, SparkFun-Capacitors:0805
- added SJ3, SJ4, SJ5: SOLDERJUMPERTRACE, SparkFun-Passives:SJ_2S-TRACE
- C1: device SparkFun-Capacitors:1206 -> SparkFun-Capacitors:1210
- moved LOGO3 7.00 mm to (48.0, 33.9)
Connections:
- net +5V: now also SJ3.1, SJ3.2; no longer C8.1, C8.2
- net GND: now also SJ5.1, SJ5.2; no longer C7.1, C7.2
- net VCC: now also SJ4.1, SJ4.2; no longer C6.1, C6.2
Other:
- board text added: "MP3 Trigger Pro"
- board text removed: "MP3 Trigger"
Changed lines of the file:
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@@
 <text x="35.052" y="0.508" size="0.8128" layer="21" font="vector" ratio="15" rot="R90">Triggers</text>
 <text x="7.112" y="0.508" size="0.8128" layer="21" font="vector" ratio="15" rot="R90">Triggers</text>
-<text x="23.241" y="34.544" size="1.778" layer="21" font="vector" ratio="15">MP3 Trigger</text>
-<text x="25.4" y="31.75" size="1.778" layer="21" font="vector" ratio="15">robertsonics</text>
+<text x="21.717" y="35.687" size="1.778" layer="21" font="vector" ratio="15">MP3 Trigger Pro</text>
+<text x="24.511" y="33.147" size="1.778" layer="21" font="vector" ratio="15">robertsonics</text>
 <text x="48.26" y="-11.43" size="1.778" layer="25" font="vector" ratio="15">Jamie Robertson, Jordan McConnell</text>
 <text x="51.181" y="11.938" size="0.8128" layer="21" font="vector" ratio="15">LED</text>
@@
 <attribute name="PROD_ID" value="CAP-08064" x="26.67" y="53.34" size="1.778" layer="27" rot="R180" display="off"/>
 </element>
-<element name="C1" library="SparkFun-Capacitors" package="1206" value="10uF" x="16.51" y="54.61"/>
+<element name="C1" library="SparkFun-Capacitors" package="1210" value="10uF" x="16.51" y="54.61">
+<attribute name="PROD_ID" value="CAP-09824" x="16.51" y="54.61" size="1.778" layer="27" display="off"/>
+<attribute name="VALUE" value="10uF" x="16.51" y="54.61" size="1.778" layer="27" display="off"/>
+</element>
 <element name="C9" library="SparkFun-Capacitors" package="0603-CAP" value="0.1uF" x="43.307" y="12.319" rot="R90"/>
 <element name="C11" library="SparkFun-Capacitors" package="0603-CAP" value="1uF" x="22.86" y="39.37" rot="R180"/>
@@
 <element name="R48" library="SparkFun-Passives" package="0603-RES" value="10K" x="5.461" y="8.89" rot="R90"/>
 <element name="J8" library="SparkFun-Connectors" package="1X04" value="" x="62.23" y="24.13" rot="R90"/>
-<element name="C6" library="SparkFun-Capacitors" package="0805" value="3.3V jumper" x="30.988" y="54.991">
-<attribute name="PROD_ID" value="CAP-08064" x="30.988" y="54.991" size="1.778" layer="27" font="vector" ratio="15" display="off"/>
-</element>
-<element name="C7" library="SparkFun-Capacitors" package="0805" value="GND jumper" x="30.988" y="56.769">
-<attribute name="PROD_ID" value="CAP-08064" x="30.988" y="56.769" size="1.778" layer="27" font="vector" ratio="15" display="off"/>
-</element>
-<element name="C8" library="SparkFun-Capacitors" package="0805" value="5V jumper" x="30.988" y="53.213">
-<attribute name="PROD_ID" value="CAP-08064" x="30.988" y="53.213" size="1.778" layer="27" font="vector" ratio="15" display="off"/>
-</element>
 <element name="SJ1" library="SparkFun-Passives" package="SJ_2S-TRACE" value="SOLDERJUMPERTRACE" x="45.72" y="55.88"/>
 <element name="SJ2" library="SparkFun-Passives" package="SJ_2S-NO" value="SOLDERJUMPERNO" x="60.833" y="36.703" rot="R90"/>
@@
 <element name="LOGO1" library="SparkFun-Aesthetics" package="OSHW-LOGO-L" value="OSHW-LOGOL" x="31.75" y="3.302" rot="MR0"/>
 <element name="LOGO2" library="SparkFun-Aesthetics" package="SFE-NEW-WEBLOGO" value="LOGO-SFENEW" x="40.64" y="30.48" rot="MR0"/>
-<element name="LOGO3" library="SparkFun-Aesthetics" package="SFE-LOGO-FLAME" value="LOGO-SFESK" x="41.021" y="34.417"/>
+<element name="LOGO3" library="SparkFun-Aesthetics" package="SFE-LOGO-FLAME" value="LOGO-SFESK" x="48.006" y="33.909"/>
+<element name="SJ3" library="SparkFun-Passives" package="SJ_2S-TRACE" value="SOLDERJUMPERTRACE" x="31.115" y="53.213"/>
+<element name="SJ4" library="SparkFun-Passives" package="SJ_2S-TRACE" value="SOLDERJUMPERTRACE" x="31.115" y="54.991" rot="R180"/>
+<element name="SJ5" library="SparkFun-Passives" package="SJ_2S-TRACE" value="SOLDERJUMPERTRACE" x="31.115" y="56.769"/>
 </elements>
 <signals>
@@
 <wire x1="3.81" y1="51.42" x2="5.7" y2="51.42" width="0.254" layer="1"/>
 <wire x1="5.7" y1="51.42" x2="8.89" y2="54.61" width="0.254" layer="1"/>
-<wire x1="8.89" y1="54.61" x2="15.11" y2="54.61" width="0.254" layer="1"/>
+<wire x1="8.89" y1="54.61" x2="14.91" y2="54.61" width="0.254" layer="1"/>
 <wire x1="22.1488" y1="49.3014" x2="22.1488" y2="50.2412" width="0.254" layer="1"/>
 <wire x1="22.1488" y1="50.2412" x2="21.59" y2="50.8" width="0.254" layer="1"/>
 <wire x1="21.59" y1="50.8" x2="16.51" y2="50.8" width="0.254" layer="1"/>
-<wire x1="16.51" y1="50.8" x2="15.24" y2="52.07" width="0.254" layer="1"/>
-<wire x1="15.24" y1="52.07" x2="15.24" y2="54.48" width="0.254" layer="1"/>
-<wire x1="15.24" y1="54.48" x2="15.11" y2="54.61" width="0.254" layer="1"/>
+<wire x1="16.51" y1="50.8" x2="14.91" y2="52.4" width="0.254" layer="1"/>
+<wire x1="15.24" y1="54.48" x2="14.91" y2="54.61" width="0.254" layer="1"/>
+<wire x1="14.91" y1="52.4" x2="14.91" y2="54.61" width="0.254" layer="1"/>
 </signal>
 <signal name="GND">
@@
 <vertex x="63.5" y="58.42"/>
 </polygon>
-<contactref element="C7" pad="1"/>
-<contactref element="C7" pad="2"/>
 <contactref element="J6" pad="1"/>
 <contactref element="J6" pad="15"/>
@@
 <wire x1="35.56" y1="55.46" x2="34.583" y2="55.46" width="0.254" layer="1"/>
 <wire x1="34.583" y1="55.46" x2="33.274" y2="56.769" width="0.254" layer="1"/>
-<wire x1="33.274" y1="56.769" x2="31.888" y2="56.769" width="0.254" layer="1"/>
 <wire x1="27.57" y1="55.88" x2="28.194" y2="55.88" width="0.254" layer="1"/>
 <wire x1="28.194" y1="55.88" x2="29.083" y2="56.769" width="0.254" layer="1"/>
-<wire x1="29.083" y1="56.769" x2="30.088" y2="56.769" width="0.254" layer="1"/>
-<wire x1="30.088" y1="56.769" x2="31.888" y2="56.769" width="0.254" layer="1"/>
 <via x="33.528" y="19.685" extent="1-16" drill="0.254"/>
 <via x="30.353" y="22.606" extent="1-16" drill="0.254"/>
@@
 <wire x1="37.2436" y1="19.84" x2="33.683" y2="19.84" width="0.2032" layer="1"/>
 <wire x1="33.683" y1="19.84" x2="33.528" y2="19.685" width="0.2032" layer="1"/>
+<contactref element="SJ5" pad="1"/>
+<contactref element="SJ5" pad="2"/>
+<wire x1="33.274" y1="56.769" x2="31.623" y2="56.769" width="0.254" layer="1"/>
+<wire x1="29.083" y1="56.769" x2="30.607" y2="56.769" width="0.254" layer="1"/>
+<wire x1="30.607" y1="56.769" x2="31.623" y2="56.769" width="0.254" layer="1"/>
 </signal>
 <signal name="+5V">
@@
 <contactref element="C31" pad="2"/>
 <contactref element="J8" pad="4"/>
-<contactref element="C8" pad="2"/>
-<contactref element="C8" pad="1"/>
 <contactref element="SJ2" pad="2"/>
 <wire x1="58.745" y1="50.4167" x2="58.745" y2="51.379" width="0.254" layer="1"/>
@@
 <wire x1="23.76" y1="55.51" x2="24.13" y2="55.88" width="0.254" layer="1"/>
 <wire x1="24.13" y1="55.88" x2="25.77" y2="55.88" width="0.254" layer="1"/>
-<wire x1="30.088" y1="53.213" x2="29.591" y2="53.213" width="0.254" layer="1"/>
 <wire x1="29.591" y1="53.213" x2="29.083" y2="52.705" width="0.254" layer="1"/>
 <wire x1="29.083" y1="52.705" x2="29.083" y2="51.181" width="0.254" layer="1"/>
@@
 <wire x1="27.686" y1="50.546" x2="27.686" y2="49.6261" width="0.254" layer="1"/>
 <wire x1="27.686" y1="49.6261" x2="27.62" y2="49.5601" width="0.254" layer="1"/>
-<wire x1="30.088" y1="53.213" x2="31.888" y2="53.213" width="0.254" layer="1"/>
 <wire x1="22.1488" y1="46.99" x2="15.951" y2="46.99" width="0.254" layer="1"/>
 <wire x1="57.531" y1="52.578" x2="57.277" y2="52.324" width="0.254" layer="1"/>
@@
 <via x="33.655" y="52.197" extent="1-16" drill="0.508"/>
 <wire x1="33.655" y1="52.197" x2="32.639" y2="53.213" width="0.254" layer="1"/>
-<wire x1="32.639" y1="53.213" x2="31.888" y2="53.213" width="0.254" layer="1"/>
+<contactref element="SJ3" pad="2"/>
+<contactref element="SJ3" pad="1"/>
+<wire x1="29.591" y1="53.213" x2="30.607" y2="53.213" width="0.254" layer="1"/>
+<wire x1="32.639" y1="53.213" x2="31.623" y2="53.213" width="0.254" layer="1"/>
+<wire x1="30.607" y1="53.213" x2="31.623" y2="53.213" width="0.254" layer="1"/>
 </signal>
 <signal name="N$2">
@@
 <contactref element="R48" pad="2"/>
 <contactref element="J8" pad="3"/>
-<contactref element="C6" pad="2"/>
-<contactref element="C6" pad="1"/>
 <contactref element="R28" pad="2"/>
 <contactref element="R25" pad="2"/>
@@
 <wire x1="35.56" y1="53.76" x2="34.886" y2="53.76" width="0.254" layer="1"/>
 <wire x1="34.886" y1="53.76" x2="33.655" y2="54.991" width="0.254" layer="1"/>
-<wire x1="33.655" y1="54.991" x2="31.888" y2="54.991" width="0.254" layer="1"/>
 <wire x1="36.475" y1="48.62" x2="36.475" y2="51.155" width="0.254" layer="1"/>
 <wire x1="36.475" y1="51.155" x2="35.56" y2="52.07" width="0.254" layer="1"/>
@@
 <wire x1="41.025" y1="46.097" x2="40.513" y2="46.609" width="0.254" layer="1"/>
 <wire x1="33.02" y1="46.14" x2="33.02" y2="44.03" width="0.254" layer="1"/>
-<wire x1="30.088" y1="54.991" x2="29.337" y2="54.991" width="0.254" layer="1"/>
 <wire x1="29.337" y1="54.991" x2="28.956" y2="54.61" width="0.254" layer="1"/>
 <wire x1="28.956" y1="54.61" x2="28.956" y2="53.975" width="0.254" layer="1"/>
 <wire x1="28.956" y1="53.975" x2="28.321" y2="53.34" width="0.254" layer="1"/>
 <wire x1="28.321" y1="53.34" x2="27.57" y2="53.34" width="0.254" layer="1"/>
-<wire x1="30.088" y1="54.991" x2="31.888" y2="54.991" width="0.254" layer="1"/>
 <wire x1="27.62" y1="45.532" x2="27.94" y2="45.212" width="0.254" layer="1"/>
 <wire x1="27.94" y1="45.212" x2="27.94" y2="44.03" width="0.254" layer="1"/>
@@
 <wire x1="41.402" y1="17.78" x2="40.43" y2="16.808" width="0.254" layer="1"/>
 <wire x1="40.43" y1="16.808" x2="40.43" y2="15.679" width="0.254" layer="1"/>
+<contactref element="SJ4" pad="2"/>
+<contactref element="SJ4" pad="1"/>
+<wire x1="33.655" y1="54.991" x2="31.623" y2="54.991" width="0.254" layer="1"/>
+<wire x1="30.607" y1="54.991" x2="29.337" y2="54.991" width="0.254" layer="1"/>
+<wire x1="30.607" y1="54.991" x2="31.623" y2="54.991" width="0.254" layer="1"/>
 </signal>
 <signal name="N$3">
