File: hardware/wavtrigger.sch (EAGLE design)
At the start: 110 parts, among them J1 5.5x2.1mm Barrel, J3 USD-SOCKETNEW, J6 M08X2, J7 M08X2, U2 MIC5323-3.3, U4 STM32F405RG, U5 PCM5100, U6 LM4990, Y1 8MHz

Commit message: v11 rev for review
Parts:
- removed LOGO3: LOGO-SFESK, SparkFun-Aesthetics:LOGO-SFESK
- added C6: .39uF, SparkFun-Capacitors:CAP0603-CAP
- added J10: (no value), SparkFun-Connectors:M04PTH
- added LOGO4: SFE_LOGO_FLAME.2_INCH, SparkFun-Aesthetics:SFE_LOGO_FLAME.2_INCH
- added TP1: TEST-POINTTP_15TH_THRU, SparkFun-Passives:TEST-POINTTP_15TH_THRU
- J5, J9: value (none) -> M02PTH
Connections:
- new net I2S_DI: J10.2, U4.PB14/I2S2_XD
- new net N$21: C6.1, R9.1
- new net N$22: TP1.1, U4.PC15
- net I2S_BCLK: now also J10.3
- net I2S_LRCK: now also J10.4
- net I2S_MCLK: now also J10.1
- net LOUTL: now also C6.2; no longer R9.1
Other:
- note added: "v11"
Changed lines of the file:
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@@
 <layer number="108" name="tplace-old" color="10" fill="1" visible="yes" active="yes"/>
 <layer number="109" name="ref-old" color="11" fill="1" visible="yes" active="yes"/>
+<layer number="110" name="fp0" color="7" fill="1" visible="yes" active="yes"/>
+<layer number="111" name="LPC17xx" color="7" fill="1" visible="yes" active="yes"/>
+<layer number="112" name="tSilk" color="7" fill="1" visible="yes" active="yes"/>
+<layer number="113" name="IDFDebug" color="4" fill="1" visible="yes" active="yes"/>
 <layer number="116" name="Patch_BOT" color="9" fill="4" visible="no" active="yes"/>
 <layer number="121" name="_tsilk" color="7" fill="1" visible="no" active="yes"/>
 <layer number="122" name="_bsilk" color="7" fill="1" visible="no" active="yes"/>
+<layer number="123" name="tTestmark" color="7" fill="1" visible="yes" active="yes"/>
+<layer number="124" name="bTestmark" color="7" fill="1" visible="yes" active="yes"/>
 <layer number="125" name="_tNames" color="7" fill="1" visible="no" active="yes"/>
+<layer number="126" name="_bNames" color="7" fill="1" visible="yes" active="yes"/>
+<layer number="127" name="_tValues" color="7" fill="1" visible="yes" active="yes"/>
+<layer number="128" name="_bValues" color="7" fill="1" visible="yes" active="yes"/>
+<layer number="131" name="tAdjust" color="7" fill="1" visible="yes" active="yes"/>
+<layer number="132" name="bAdjust" color="7" fill="1" visible="yes" active="yes"/>
 <layer number="144" name="Drill_legend" color="7" fill="1" visible="no" active="yes"/>
 <layer number="151" name="HeatSink" color="7" fill="1" visible="no" active="yes"/>
+<layer number="152" name="_bDocu" color="7" fill="1" visible="yes" active="yes"/>
 <layer number="199" name="Contour" color="7" fill="1" visible="no" active="yes"/>
 <layer number="200" name="200bmp" color="1" fill="10" visible="no" active="yes"/>
@@
 <layer number="223" name="223bmp" color="24" fill="1" visible="no" active="no"/>
 <layer number="224" name="224bmp" color="25" fill="1" visible="no" active="no"/>
+<layer number="248" name="Housing" color="7" fill="1" visible="yes" active="yes"/>
+<layer number="249" name="Edge" color="7" fill="1" visible="yes" active="yes"/>
 <layer number="250" name="Descript" color="3" fill="1" visible="no" active="no"/>
 <layer number="251" name="SMDround" color="12" fill="11" visible="no" active="no"/>
@@
 <part name="LOGO1" library="SparkFun-Aesthetics" deviceset="OSHW-LOGO" device="L"/>
 <part name="LOGO2" library="SparkFun-Aesthetics" deviceset="LOGO-SFE" device="NEW"/>
-<part name="LOGO3" library="SparkFun-Aesthetics" deviceset="LOGO-SFE" device="SK"/>
 <part name="SJ3" library="SparkFun-Passives" deviceset="SOLDERJUMPER" device="TRACE"/>
 <part name="SJ4" library="SparkFun-Passives" deviceset="SOLDERJUMPER" device="TRACE"/>
@@
 <part name="FID1" library="SparkFun-Aesthetics" deviceset="FIDUCIAL" device="UFIDUCIAL"/>
 <part name="FID2" library="SparkFun-Aesthetics" deviceset="FIDUCIAL" device="UFIDUCIAL"/>
+<part name="C6" library="SparkFun-Capacitors" deviceset="CAP" device="0603-CAP" value=".39uF"/>
+<part name="TP1" library="SparkFun-Passives" deviceset="TEST-POINT" device="TP_15TH_THRU"/>
+<part name="J10" library="SparkFun-Connectors" deviceset="M04" device="PTH"/>
+<part name="LOGO4" library="SparkFun-Aesthetics" deviceset="SFE_LOGO_FLAME" device=".2_INCH"/>
 </parts>
 <sheets>
@@
 <text x="45.72" y="238.76" size="1.778" layer="96">LM1117</text>
 <text x="15.24" y="254" size="1.27" layer="97">Vin: 6V-20V</text>
+<text x="421.64" y="7.62" size="1.778" layer="94">v11</text>
 </plain>
 <instances>
@@
 <instance part="LOGO1" gate="G$1" x="297.18" y="22.86"/>
 <instance part="LOGO2" gate="G$1" x="322.58" y="17.78"/>
-<instance part="LOGO3" gate="G$1" x="322.58" y="25.4"/>
 <instance part="SJ3" gate="1" x="17.78" y="154.94" smashed="yes">
 <attribute name="NAME" x="15.24" y="157.48" size="1.778" layer="95"/>
@@
 <instance part="FID1" gate="G$1" x="358.14" y="38.1"/>
 <instance part="FID2" gate="G$1" x="363.22" y="38.1"/>
+<instance part="C6" gate="G$1" x="149.86" y="111.76" rot="R90"/>
+<instance part="TP1" gate="G$1" x="248.92" y="121.92" smashed="yes" rot="R90">
+<attribute name="NAME" x="246.38" y="119.38" size="1.778" layer="95" rot="R90"/>
+</instance>
+<instance part="J10" gate="G$1" x="391.16" y="53.34"/>
+<instance part="LOGO4" gate="G$1" x="419.1" y="35.56"/>
 </instances>
 <busses>
@@
 </segment>
 <segment>
-<pinref part="R9" gate="G$1" pin="1"/>
-<wire x1="142.24" y1="111.76" x2="144.78" y2="111.76" width="0.1524" layer="91"/>
-<label x="144.78" y="111.76" size="1.27" layer="95" xref="yes"/>
+<wire x1="152.4" y1="111.76" x2="154.94" y2="111.76" width="0.1524" layer="91"/>
+<label x="154.94" y="111.76" size="1.27" layer="95" xref="yes"/>
+<pinref part="C6" gate="G$1" pin="2"/>
 </segment>
 </net>
@@
 <label x="337.82" y="58.42" size="1.27" layer="95" xref="yes"/>
 </segment>
+<segment>
+<pinref part="J10" gate="G$1" pin="1"/>
+<wire x1="396.24" y1="50.8" x2="398.78" y2="50.8" width="0.1524" layer="91"/>
+<label x="398.78" y="50.8" size="1.27" layer="95" xref="yes"/>
+</segment>
 </net>
 <net name="I2S_BCLK" class="0">
@@
 <label x="337.82" y="50.8" size="1.27" layer="95" xref="yes"/>
 </segment>
+<segment>
+<pinref part="J10" gate="G$1" pin="3"/>
+<wire x1="396.24" y1="55.88" x2="398.78" y2="55.88" width="0.1524" layer="91"/>
+<label x="398.78" y="55.88" size="1.27" layer="95" xref="yes"/>
+</segment>
 </net>
 <net name="I2S_DOUT" class="0">
@@
 <wire x1="325.12" y1="48.26" x2="337.82" y2="48.26" width="0.1524" layer="91"/>
 <label x="337.82" y="48.26" size="1.27" layer="95" xref="yes"/>
+</segment>
+<segment>
+<pinref part="J10" gate="G$1" pin="4"/>
+<wire x1="396.24" y1="58.42" x2="398.78" y2="58.42" width="0.1524" layer="91"/>
+<label x="398.78" y="58.42" size="1.27" layer="95" xref="yes"/>
 </segment>
 </net>
@@
 <segment>
 <pinref part="U6" gate="G$1" pin="SHTDN"/>
-<wire x1="144.78" y1="119.38" x2="121.92" y2="119.38" width="0.1524" layer="91"/>
+<wire x1="127" y1="119.38" x2="121.92" y2="119.38" width="0.1524" layer="91"/>
 <pinref part="R8" gate="G$1" pin="2"/>
 <wire x1="121.92" y1="119.38" x2="116.84" y2="119.38" width="0.1524" layer="91"/>
 <wire x1="121.92" y1="119.38" x2="121.92" y2="124.46" width="0.1524" layer="91"/>
 <junction x="121.92" y="119.38"/>
-<label x="144.78" y="119.38" size="1.27" layer="95" xref="yes"/>
+<label x="127" y="119.38" size="1.27" layer="95" xref="yes"/>
 </segment>
 <segment>
@@
 </segment>
 </net>
+<net name="N$21" class="0">
+<segment>
+<pinref part="R9" gate="G$1" pin="1"/>
+<pinref part="C6" gate="G$1" pin="1"/>
+<wire x1="142.24" y1="111.76" x2="144.78" y2="111.76" width="0.1524" layer="91"/>
+</segment>
+</net>
+<net name="N$22" class="0">
+<segment>
+<pinref part="TP1" gate="G$1" pin="1"/>
+<wire x1="248.92" y1="121.92" x2="248.92" y2="119.38" width="0.1524" layer="91"/>
+<pinref part="U4" gate="G$1" pin="PC15"/>
+<wire x1="248.92" y1="119.38" x2="266.7" y2="119.38" width="0.1524" layer="91"/>
+</segment>
+</net>
+<net name="I2S_DI" class="0">
+<segment>
+<pinref part="J10" gate="G$1" pin="2"/>
+<wire x1="396.24" y1="53.34" x2="398.78" y2="53.34" width="0.1524" layer="91"/>
+<label x="398.78" y="53.34" size="1.27" layer="95" xref="yes"/>
+</segment>
+<segment>
+<pinref part="U4" gate="G$1" pin="PB14/I2S2_XD"/>
+<wire x1="325.12" y1="53.34" x2="337.82" y2="53.34" width="0.1524" layer="91"/>
+<label x="337.82" y="53.34" size="1.27" layer="95" xref="yes"/>
+</segment>
+</net>
