File: hardware/wavtrigger.sch (EAGLE design)
At the start: 113 parts, among them J1 5.5x2.1mm Barrel, J3 USD-SOCKETNEW, J5 M02PTH, J6 M08X2, J7 M08X2, J9 M02PTH, U2 MIC5323-3.3, U4 STM32F405RG, U5 PCM5100, U6 LM4990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

Commit message: added regular fiducial, changed barrel jack FP
Parts:
- FID1, FID2: value FIDUCIALUFIDUCIAL -> FIDUCIAL1X2; device SparkFun-Aesthetics:FIDUCIALUFIDUCIAL -> SparkFun-Aesthetics:FIDUCIAL1X2
- J1: device SparkFun-Connectors:POWER_JACKSMD -> Testing:POWER_JACKOVERPASTE_REDBOARD_0603
Changed lines of the file:
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@@
 <layer number="54" name="bGND_GNDA" color="1" fill="9" visible="no" active="no"/>
 <layer number="56" name="wert" color="7" fill="1" visible="no" active="no"/>
+<layer number="57" name="tCAD" color="7" fill="1" visible="no" active="no"/>
 <layer number="91" name="Nets" color="2" fill="1" visible="yes" active="yes"/>
 <layer number="92" name="Busses" color="1" fill="1" visible="yes" active="yes"/>
@@
 <layer number="97" name="Info" color="7" fill="1" visible="yes" active="yes"/>
 <layer number="98" name="Guide" color="6" fill="1" visible="yes" active="yes"/>
+<layer number="99" name="SpiceOrder" color="7" fill="1" visible="yes" active="yes"/>
 <layer number="100" name="Muster" color="7" fill="1" visible="no" active="no"/>
 <layer number="101" name="Patch_Top" color="12" fill="4" visible="no" active="yes"/>
@@
 <layer number="132" name="bAdjust" color="7" fill="1" visible="yes" active="yes"/>
 <layer number="144" name="Drill_legend" color="7" fill="1" visible="no" active="yes"/>
+<layer number="150" name="Notes" color="7" fill="1" visible="yes" active="yes"/>
 <layer number="151" name="HeatSink" color="7" fill="1" visible="no" active="yes"/>
 <layer number="152" name="_bDocu" color="7" fill="1" visible="yes" active="yes"/>
+<layer number="153" name="FabDoc1" color="7" fill="1" visible="yes" active="yes"/>
+<layer number="154" name="FabDoc2" color="7" fill="1" visible="yes" active="yes"/>
+<layer number="155" name="FabDoc3" color="7" fill="1" visible="yes" active="yes"/>
 <layer number="199" name="Contour" color="7" fill="1" visible="no" active="yes"/>
 <layer number="200" name="200bmp" color="1" fill="10" visible="no" active="yes"/>
@@
 </classes>
 <parts>
-<part name="J1" library="SparkFun-Connectors" deviceset="POWER_JACK" device="SMD" value="5.5x2.1mm Barrel"/>
+<part name="J1" library="Testing" deviceset="POWER_JACK" device="OVERPASTE_REDBOARD_0603" value="5.5x2.1mm Barrel"/>
 <part name="GND1" library="supply1" deviceset="GND" device=""/>
 <part name="GND2" library="supply1" deviceset="GND" device=""/>
@@
 <part name="GND34" library="supply1" deviceset="GND" device=""/>
 <part name="FRAME2" library="SparkFun-Aesthetics" deviceset="FRAME-LEDGER" device=""/>
-<part name="FID1" library="SparkFun-Aesthetics" deviceset="FIDUCIAL" device="UFIDUCIAL"/>
-<part name="FID2" library="SparkFun-Aesthetics" deviceset="FIDUCIAL" device="UFIDUCIAL"/>
 <part name="C6" library="SparkFun-Capacitors" deviceset="CAP" device="0603-CAP" value=".39uF"/>
 <part name="TP1" library="SparkFun-Passives" deviceset="TEST-POINT" device="TP_15TH_THRU"/>
 <part name="J10" library="SparkFun-Connectors" deviceset="M04" device="PTH"/>
 <part name="LOGO4" library="SparkFun-Aesthetics" deviceset="SFE_LOGO_FLAME" device=".2_INCH"/>
+<part name="FID1" library="SparkFun-Aesthetics" deviceset="FIDUCIAL" device="1X2"/>
+<part name="FID2" library="SparkFun-Aesthetics" deviceset="FIDUCIAL" device="1X2"/>
 </parts>
 <sheets>
@@
 <instance part="FRAME2" gate="G$1" x="0" y="0"/>
 <instance part="FRAME2" gate="G$2" x="330.2" y="0"/>
-<instance part="FID1" gate="G$1" x="358.14" y="38.1"/>
-<instance part="FID2" gate="G$1" x="363.22" y="38.1"/>
 <instance part="C6" gate="G$1" x="149.86" y="111.76" rot="R90"/>
 <instance part="TP1" gate="G$1" x="248.92" y="121.92" smashed="yes" rot="R90">
@@
 <instance part="J10" gate="G$1" x="391.16" y="53.34"/>
 <instance part="LOGO4" gate="G$1" x="419.1" y="35.56"/>
+<instance part="FID1" gate="G$1" x="365.76" y="38.1"/>
+<instance part="FID2" gate="G$1" x="373.38" y="38.1"/>
 </instances>
 <busses>
