File: hardware/wavtrigger.sch (EAGLE design)
At the start: 105 parts, among them J1 5.5x2.1mm Barrel, J3 USD-SOCKETNEW, J6 M08X2, J7 M08X2, U1 NCP1117, U2 MIC5323-3.3, U4 STM32F405RG, U5 PCM5100, U6 LM4990, Y1 8MHz

Commit message: v04 hardware files
Parts:
- removed JP1: (no value), SparkFun-Connectors:M03PTH
- removed SJ1: SOLDERJUMPERTRACE, SparkFun-Passives:SOLDERJUMPERTRACE
- removed U1: NCP1117, SparkFun-PowerIC:V_REG_LM1117SOT223
- added S1: (no value), SparkFun-Electromechanical:SWITCH-SPDT-SMD-A
- added S2: SWITCH-MOMENTARY-2SMD, SparkFun-Electromechanical:SWITCH-MOMENTARY-2SMD
- added U3: MIC5219 5V, SparkFun-PowerIC:V_REG_MIC52195V
- U4: device robertsonics:STM32F405RG -> SparkFun-DigitalIC:STM32F405RG
Connections:
- removed net AMPIN: R9.1, SJ1.2
- net +5V: now also U3.OUT; no longer U1.OUT, U1.OUT@1
- net BOOT0: now also S1.P; no longer JP1.2
- net GND: now also S2.1, U3.GND; no longer U1.ADJ
- net LOUTL: now also R9.1; no longer SJ1.1
- net N$10: now also S1.O; no longer JP1.3
- net N$7: now also S1.S; no longer JP1.1
- net TRIG00: now also S2.2
- net VIN_9V: now also U3.EN, U3.IN; no longer U1.IN
Other:
- moved on the sheet: C1

Commit message: Next round of protos ready for order, v04
Parts:
- removed U3: MIC5219 5V, SparkFun-PowerIC:V_REG_MIC52195V
- added R49: 240, SparkFun-Resistors:240OHM1/10W1%(0603)
- added R50: 715, SparkFun-Resistors:RESISTOR0603
- added U1: (no value), SparkFun-PowerIC:V_REG_LM1117SOT223
- R25, R26, R27, R28, R29, R30, R31, R32, R41, R42, R43, R44, R45, R46, R47, R48: value 10K -> DNP
Connections:
- new net BUTTON: S2.2, U4.PB1
- new net N$13: R49.2, R50.2, U1.ADJ
- net +5V: now also R49.1, U1.OUT, U1.OUT@1; no longer U3.OUT
- net GND: now also R50.1; no longer J3.SHIELD@4, U3.GND
- net SD_CD: now also J3.SHIELD@4
- net TRIG00: no longer S2.2
- net VIN_9V: now also U1.IN; no longer U3.EN, U3.IN
Other:
- note added: "LM1117"
- moved on the sheet: C1, C2, C3, C4, C5, J1, U2

Commit message: v10 red ready
Parts:
- added J9: (no value), SparkFun-Connectors:M02PTH
Connections:
- removed net VIN_9V: C1.1, J1.PWR, U1.IN
- new net VIN: C1.1, J1.PWR, J9.2, U1.IN
- net GND: now also J9.1
Other:
- note added: "Vin: 6V-20V"
- moved on the sheet: C1, C2, J1, R49, R50, U1
Changed lines of the file:
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@@
 <part name="R50" library="SparkFun-Resistors" deviceset="RESISTOR" device="0603" value="715"/>
 <part name="U1" library="SparkFun-PowerIC" deviceset="V_REG_LM1117" device="SOT223"/>
+<part name="J9" library="SparkFun-Connectors" deviceset="M02" device="PTH"/>
+<part name="GND34" library="supply1" deviceset="GND" device=""/>
 </parts>
 <sheets>
@@
 <text x="30.48" y="139.7" size="1.778" layer="95">3.3V jumper</text>
 <text x="55.88" y="139.7" size="1.778" layer="95">GND jumper</text>
-<text x="35.56" y="228.6" size="1.778" layer="96">LM1117</text>
+<text x="38.1" y="223.52" size="1.778" layer="96">LM1117</text>
+<text x="7.62" y="238.76" size="1.27" layer="97">Vin: 6V-20V</text>
 </plain>
 <instances>
 <instance part="FRAME1" gate="G$1" x="0" y="0"/>
-<instance part="J1" gate="G$1" x="20.32" y="228.6"/>
-<instance part="GND1" gate="1" x="33.02" y="205.74"/>
+<instance part="J1" gate="G$1" x="22.86" y="223.52"/>
+<instance part="GND1" gate="1" x="35.56" y="200.66"/>
 <instance part="GND2" gate="1" x="17.78" y="172.72"/>
 <instance part="U4" gate="G$1" x="271.78" y="76.2"/>
-<instance part="C2" gate="G$1" x="71.12" y="220.98"/>
-<instance part="P+1" gate="1" x="78.74" y="243.84"/>
+<instance part="C2" gate="G$1" x="73.66" y="215.9"/>
+<instance part="P+1" gate="1" x="81.28" y="238.76"/>
 <instance part="U2" gate="G$1" x="45.72" y="185.42"/>
 <instance part="C3" gate="G$1" x="17.78" y="182.88"/>
@@
 <instance part="C4" gate="G$1" x="60.96" y="172.72"/>
 <instance part="C5" gate="G$1" x="73.66" y="182.88"/>
-<instance part="GND4" gate="1" x="60.96" y="165.1"/>
+<instance part="GND4" gate="1" x="60.96" y="167.64"/>
 <instance part="GND5" gate="1" x="73.66" y="175.26"/>
 <instance part="P+4" gate="VCC" x="81.28" y="198.12"/>
-<instance part="C1" gate="G$1" x="33.02" y="220.98"/>
+<instance part="C1" gate="G$1" x="35.56" y="215.9"/>
 <instance part="C9" gate="G$1" x="233.68" y="121.92"/>
 <instance part="P+5" gate="VCC" x="233.68" y="132.08"/>
@@
 </instance>
 <instance part="GND33" gate="1" x="337.82" y="162.56"/>
-<instance part="R49" gate="G$1" x="53.34" y="226.06" rot="R180"/>
-<instance part="R50" gate="G$1" x="45.72" y="218.44" rot="R90"/>
-<instance part="U1" gate="G$1" x="45.72" y="236.22" smashed="yes">
-<attribute name="NAME" x="41.148" y="239.268" size="1.778" layer="95"/>
-<attribute name="VALUE" x="48.26" y="226.06" size="1.778" layer="96"/>
+<instance part="R49" gate="G$1" x="55.88" y="220.98" rot="R180"/>
+<instance part="R50" gate="G$1" x="48.26" y="213.36" rot="R90"/>
+<instance part="U1" gate="G$1" x="48.26" y="231.14" smashed="yes">
+<attribute name="NAME" x="43.688" y="234.188" size="1.778" layer="95"/>
+<attribute name="VALUE" x="50.8" y="220.98" size="1.778" layer="96"/>
 </instance>
+<instance part="J9" gate="G$1" x="15.24" y="246.38"/>
+<instance part="GND34" gate="1" x="25.4" y="241.3"/>
 </instances>
 <busses>
 </busses>
 <nets>
-<net name="VIN_9V" class="0">
-<segment>
-<pinref part="J1" gate="G$1" pin="PWR"/>
-<wire x1="22.86" y1="236.22" x2="33.02" y2="236.22" width="0.1524" layer="91"/>
-<wire x1="33.02" y1="226.06" x2="33.02" y2="236.22" width="0.1524" layer="91"/>
-<pinref part="C1" gate="G$1" pin="1"/>
-<pinref part="U1" gate="G$1" pin="IN"/>
-<wire x1="38.1" y1="236.22" x2="33.02" y2="236.22" width="0.1524" layer="91"/>
-<junction x="33.02" y="236.22"/>
-</segment>
-</net>
 <net name="GND" class="0">
 <segment>
 <pinref part="GND1" gate="1" pin="GND"/>
-<wire x1="33.02" y1="218.44" x2="33.02" y2="210.82" width="0.1524" layer="91"/>
-<wire x1="33.02" y1="210.82" x2="33.02" y2="208.28" width="0.1524" layer="91"/>
-<wire x1="25.4" y1="210.82" x2="33.02" y2="210.82" width="0.1524" layer="91"/>
-<junction x="33.02" y="210.82"/>
+<wire x1="35.56" y1="213.36" x2="35.56" y2="205.74" width="0.1524" layer="91"/>
+<wire x1="35.56" y1="205.74" x2="35.56" y2="203.2" width="0.1524" layer="91"/>
+<wire x1="27.94" y1="205.74" x2="35.56" y2="205.74" width="0.1524" layer="91"/>
+<junction x="35.56" y="205.74"/>
 <pinref part="C2" gate="G$1" pin="2"/>
-<wire x1="33.02" y1="210.82" x2="45.72" y2="210.82" width="0.1524" layer="91"/>
-<wire x1="45.72" y1="210.82" x2="71.12" y2="210.82" width="0.1524" layer="91"/>
-<wire x1="71.12" y1="210.82" x2="71.12" y2="218.44" width="0.1524" layer="91"/>
+<wire x1="35.56" y1="205.74" x2="48.26" y2="205.74" width="0.1524" layer="91"/>
+<wire x1="48.26" y1="205.74" x2="73.66" y2="205.74" width="0.1524" layer="91"/>
+<wire x1="73.66" y1="205.74" x2="73.66" y2="213.36" width="0.1524" layer="91"/>
 <pinref part="C1" gate="G$1" pin="2"/>
 <pinref part="J1" gate="G$1" pin="GNDBREAK"/>
-<wire x1="22.86" y1="233.68" x2="25.4" y2="233.68" width="0.1524" layer="91"/>
-<wire x1="25.4" y1="233.68" x2="25.4" y2="231.14" width="0.1524" layer="91"/>
+<wire x1="25.4" y1="228.6" x2="27.94" y2="228.6" width="0.1524" layer="91"/>
+<wire x1="27.94" y1="228.6" x2="27.94" y2="226.06" width="0.1524" layer="91"/>
 <pinref part="J1" gate="G$1" pin="GND"/>
-<wire x1="25.4" y1="231.14" x2="25.4" y2="210.82" width="0.1524" layer="91"/>
-<wire x1="22.86" y1="231.14" x2="25.4" y2="231.14" width="0.1524" layer="91"/>
-<junction x="25.4" y="231.14"/>
+<wire x1="27.94" y1="226.06" x2="27.94" y2="205.74" width="0.1524" layer="91"/>
+<wire x1="25.4" y1="226.06" x2="27.94" y2="226.06" width="0.1524" layer="91"/>
+<junction x="27.94" y="226.06"/>
 <pinref part="R50" gate="G$1" pin="1"/>
-<wire x1="45.72" y1="210.82" x2="45.72" y2="213.36" width="0.1524" layer="91"/>
-<junction x="45.72" y="210.82"/>
+<wire x1="48.26" y1="205.74" x2="48.26" y2="208.28" width="0.1524" layer="91"/>
+<junction x="48.26" y="205.74"/>
 </segment>
 <segment>
@@
 <pinref part="C4" gate="G$1" pin="2"/>
 <pinref part="GND4" gate="1" pin="GND"/>
-<wire x1="60.96" y1="167.64" x2="60.96" y2="170.18" width="0.1524" layer="91"/>
 </segment>
 <segment>
@@
 <wire x1="337.82" y1="167.64" x2="337.82" y2="165.1" width="0.1524" layer="91"/>
 </segment>
+<segment>
+<pinref part="J9" gate="G$1" pin="1"/>
+<wire x1="22.86" y1="246.38" x2="25.4" y2="246.38" width="0.1524" layer="91"/>
+<wire x1="25.4" y1="246.38" x2="25.4" y2="243.84" width="0.1524" layer="91"/>
+<pinref part="GND34" gate="1" pin="GND"/>
+</segment>
 </net>
 <net name="+5V" class="0">
 <segment>
 <pinref part="C2" gate="G$1" pin="1"/>
-<wire x1="78.74" y1="236.22" x2="71.12" y2="236.22" width="0.1524" layer="91"/>
-<wire x1="71.12" y1="236.22" x2="71.12" y2="226.06" width="0.1524" layer="91"/>
+<wire x1="81.28" y1="231.14" x2="73.66" y2="231.14" width="0.1524" layer="91"/>
+<wire x1="73.66" y1="231.14" x2="73.66" y2="220.98" width="0.1524" layer="91"/>
 <pinref part="P+1" gate="1" pin="+5V"/>
-<wire x1="78.74" y1="236.22" x2="78.74" y2="241.3" width="0.1524" layer="91"/>
+<wire x1="81.28" y1="231.14" x2="81.28" y2="236.22" width="0.1524" layer="91"/>
 <pinref part="U1" gate="G$1" pin="OUT"/>
-<wire x1="53.34" y1="236.22" x2="55.88" y2="236.22" width="0.1524" layer="91"/>
-<junction x="71.12" y="236.22"/>
+<wire x1="55.88" y1="231.14" x2="58.42" y2="231.14" width="0.1524" layer="91"/>
+<junction x="73.66" y="231.14"/>
 <pinref part="U1" gate="G$1" pin="OUT@1"/>
-<wire x1="55.88" y1="236.22" x2="60.96" y2="236.22" width="0.1524" layer="91"/>
-<wire x1="60.96" y1="236.22" x2="71.12" y2="236.22" width="0.1524" layer="91"/>
-<wire x1="53.34" y1="233.68" x2="55.88" y2="233.68" width="0.1524" layer="91"/>
-<wire x1="55.88" y1="233.68" x2="55.88" y2="236.22" width="0.1524" layer="91"/>
-<junction x="55.88" y="236.22"/>
+<wire x1="58.42" y1="231.14" x2="63.5" y2="231.14" width="0.1524" layer="91"/>
+<wire x1="63.5" y1="231.14" x2="73.66" y2="231.14" width="0.1524" layer="91"/>
+<wire x1="55.88" y1="228.6" x2="58.42" y2="228.6" width="0.1524" layer="91"/>
+<wire x1="58.42" y1="228.6" x2="58.42" y2="231.14" width="0.1524" layer="91"/>
+<junction x="58.42" y="231.14"/>
 <pinref part="R49" gate="G$1" pin="1"/>
-<wire x1="58.42" y1="226.06" x2="60.96" y2="226.06" width="0.1524" layer="91"/>
-<wire x1="60.96" y1="226.06" x2="60.96" y2="236.22" width="0.1524" layer="91"/>
-<junction x="60.96" y="236.22"/>
+<wire x1="60.96" y1="220.98" x2="63.5" y2="220.98" width="0.1524" layer="91"/>
+<wire x1="63.5" y1="220.98" x2="63.5" y2="231.14" width="0.1524" layer="91"/>
+<junction x="63.5" y="231.14"/>
 </segment>
 <segment>
@@
 <pinref part="R50" gate="G$1" pin="2"/>
 <pinref part="U1" gate="G$1" pin="ADJ"/>
-<wire x1="45.72" y1="223.52" x2="45.72" y2="226.06" width="0.1524" layer="91"/>
+<wire x1="48.26" y1="218.44" x2="48.26" y2="220.98" width="0.1524" layer="91"/>
 <pinref part="R49" gate="G$1" pin="2"/>
-<wire x1="45.72" y1="226.06" x2="45.72" y2="228.6" width="0.1524" layer="91"/>
-<wire x1="48.26" y1="226.06" x2="45.72" y2="226.06" width="0.1524" layer="91"/>
-<junction x="45.72" y="226.06"/>
+<wire x1="48.26" y1="220.98" x2="48.26" y2="223.52" width="0.1524" layer="91"/>
+<wire x1="50.8" y1="220.98" x2="48.26" y2="220.98" width="0.1524" layer="91"/>
+<junction x="48.26" y="220.98"/>
 </segment>
 </net>
@@
 </segment>
 </net>
+<net name="VIN" class="0">
+<segment>
+<pinref part="J1" gate="G$1" pin="PWR"/>
+<wire x1="25.4" y1="231.14" x2="35.56" y2="231.14" width="0.1524" layer="91"/>
+<wire x1="35.56" y1="220.98" x2="35.56" y2="231.14" width="0.1524" layer="91"/>
+<pinref part="C1" gate="G$1" pin="1"/>
+<pinref part="U1" gate="G$1" pin="IN"/>
+<wire x1="40.64" y1="231.14" x2="35.56" y2="231.14" width="0.1524" layer="91"/>
+<junction x="35.56" y="231.14"/>
+</segment>
+<segment>
+<pinref part="J9" gate="G$1" pin="2"/>
+<wire x1="22.86" y1="248.92" x2="25.4" y2="248.92" width="0.1524" layer="91"/>
+<label x="25.4" y="248.92" size="1.27" layer="95" xref="yes"/>
+</segment>
+</net>

Commit message: v10, frame update
Parts:
- removed CC_TEXT1: CREATIVE_COMMONS, SparkFun-Aesthetics:CREATIVE_COMMONS
- added FRAME2: FRAME-LEDGER, SparkFun-Aesthetics:FRAME-LEDGER
Other:
- moved on the sheet: C1, C10, C11, C12, C13, C14, C15, C16, C17, C18, C19, C2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

Commit message: Added local micro fiducials
Parts:
- added FID1, FID2: FIDUCIALUFIDUCIAL, SparkFun-Aesthetics:FIDUCIALUFIDUCIAL
Changed lines of the file:
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@@
 <part name="GND34" library="supply1" deviceset="GND" device=""/>
 <part name="FRAME2" library="SparkFun-Aesthetics" deviceset="FRAME-LEDGER" device=""/>
+<part name="FID1" library="SparkFun-Aesthetics" deviceset="FIDUCIAL" device="UFIDUCIAL"/>
+<part name="FID2" library="SparkFun-Aesthetics" deviceset="FIDUCIAL" device="UFIDUCIAL"/>
 </parts>
 <sheets>
@@
 <instance part="FRAME2" gate="G$1" x="0" y="0"/>
 <instance part="FRAME2" gate="G$2" x="330.2" y="0"/>
+<instance part="FID1" gate="G$1" x="358.14" y="38.1"/>
+<instance part="FID2" gate="G$1" x="363.22" y="38.1"/>
 </instances>
 <busses>

Commit message: updated v10, changed C24-25 values to improve audio quality
Parts:
- C24, C25: value 0.1uF -> 2.2uF
Changed lines of the file:
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@@
 <part name="C22" library="SparkFun-Capacitors" deviceset="CAP" device="0603-CAP" value="0.1uF"/>
 <part name="C23" library="SparkFun-Capacitors" deviceset="CAP" device="0603-CAP" value="0.1uF"/>
-<part name="C24" library="SparkFun-Capacitors" deviceset="CAP" device="0603-CAP" value="0.1uF"/>
+<part name="C24" library="SparkFun-Capacitors" deviceset="CAP" device="0603-CAP" value="2.2uF"/>
 <part name="P+10" library="supply1" deviceset="VCC" device="" value="+3V3"/>
 <part name="GND21" library="supply1" deviceset="GND" device=""/>
 <part name="GND22" library="supply1" deviceset="GND" device=""/>
-<part name="C25" library="SparkFun-Capacitors" deviceset="CAP" device="0603-CAP" value="0.1uF"/>
+<part name="C25" library="SparkFun-Capacitors" deviceset="CAP" device="0603-CAP" value="2.2uF"/>
 <part name="C26" library="SparkFun-Capacitors" deviceset="CAP" device="0603-CAP" value="0.1uF"/>
 <part name="C27" library="SparkFun-Capacitors" deviceset="CAP" device="0603-CAP" value="10uF"/>

Commit message: changed micro fid to regular
also deleted "wrong" panel, re-doing it
Parts:
- FID1, FID2: value FIDUCIALUFIDUCIAL -> FIDUCIAL1X2; device SparkFun-Aesthetics:FIDUCIALUFIDUCIAL -> SparkFun-Aesthetics:FIDUCIAL1X2
Changed lines of the file:
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@@
 <?xml version="1.0" encoding="utf-8"?>
 <!DOCTYPE eagle SYSTEM "eagle.dtd">
-<eagle version="6.5.0">
+<eagle version="6.6.0">
 <drawing>
 <settings>
@@
 <part name="GND34" library="supply1" deviceset="GND" device=""/>
 <part name="FRAME2" library="SparkFun-Aesthetics" deviceset="FRAME-LEDGER" device=""/>
-<part name="FID1" library="SparkFun-Aesthetics" deviceset="FIDUCIAL" device="UFIDUCIAL"/>
-<part name="FID2" library="SparkFun-Aesthetics" deviceset="FIDUCIAL" device="UFIDUCIAL"/>
+<part name="FID1" library="SparkFun-Aesthetics" deviceset="FIDUCIAL" device="1X2"/>
+<part name="FID2" library="SparkFun-Aesthetics" deviceset="FIDUCIAL" device="1X2"/>
 </parts>
 <sheets>
@@
 <instance part="FRAME2" gate="G$1" x="0" y="0"/>
 <instance part="FRAME2" gate="G$2" x="330.2" y="0"/>
-<instance part="FID1" gate="G$1" x="358.14" y="38.1"/>
-<instance part="FID2" gate="G$1" x="363.22" y="38.1"/>
+<instance part="FID1" gate="G$1" x="373.38" y="38.1"/>
+<instance part="FID2" gate="G$1" x="378.46" y="38.1"/>
 </instances>
 <busses>
