File: hardware/wavtrigger.brd (EAGLE design)
At the start: 63.5 x 58.4 mm, 113 parts, among them J1 5.5x2.1mm Barrel, J3 USD-SOCKETNEW, J5 M02PTH, J6 M08X2, J7 M08X2, J9 M02PTH, U2 MIC5323-3.3, U4 STM32F405RG, U5 PCM5100, U6 LM4990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

Commit message: added regular fiducial, changed barrel jack FP
Parts:
- FID1, FID2: value FIDUCIALUFIDUCIAL -> FIDUCIAL1X2; device SparkFun-Aesthetics:MICRO-FIDUCIAL -> SparkFun-Aesthetics:FIDUCIAL-1X2
- J1: device SparkFun-Connectors:POWER_JACK_SMD -> Testing:POWER_JACK_SMD_OVERPASTE_REDBOARD_0603
- moved FID1 4.06 mm to (5.08, 52.8)
