File: hardware/wavtrigger.brd (EAGLE design)
At the start: 63.5 x 58.4 mm, 105 parts, among them J1 5.5x2.1mm Barrel, J3 USD-SOCKETNEW, J6 M08X2, J7 M08X2, U1 NCP1117, U2 MIC5323-3.3, U4 STM32F405RG, U5 PCM5100, U6 LM4990, Y1 8MHz

Commit message: v04 hardware files
Parts:
- removed JP1: (no value), SparkFun-Connectors:1X03
- removed SJ1: SOLDERJUMPERTRACE, SparkFun-Passives:SJ_2S-TRACE
- removed U1: NCP1117, SparkFun-PowerIC:SOT223
- added S1: (no value), SparkFun-Electromechanical:SWITCH-SPST-SMD-A
- added S2: SWITCH-MOMENTARY-2SMD, SparkFun-Electromechanical:TACTILE_SWITCH_SMD
- added U3: MIC5219 5V, SparkFun-PowerIC:SOT23-5
- U4: device robertsonics:TQFP-10X10-64 -> SparkFun-DigitalIC:TQFP64
- moved R40 21.1 mm to (23.6, 16.1), turned to 0 degrees
- moved R16 17.8 mm to (19.1, 55.9)
- moved R48 15.8 mm to (19.6, 16.1), turned to 180 degrees
- moved C2 10.2 mm to (22.9, 43.2), turned to 270 degrees
- moved C21 6.48 mm to (43.2, 54.6), turned to 270 degrees
- moved C28 6.48 mm to (44.5, 48.3), turned to 0 degrees
- moved C1 4.90 mm to (19.1, 50.4), turned to 90 degrees
- moved C3 4.58 mm to (22.9, 53.3), turned to 180 degrees
- moved J8 1.27 mm to (62.2, 25.4)
- turned U4 to 270 degrees
Connections:
- removed net AMPIN: R9.1, SJ1.2
- net +5V: now also U3.5; no longer U1.2, U1.4
- net AMPENA: now also U4.11; no longer U4.P$11
- net BOOT0: now also S1.2, U4.60; no longer JP1.2, U4.P$60
- net DEMP: now also U4.10; no longer U4.P$10
- net FILTER: now also U4.9; no longer U4.P$9
- net GND: now also S2.1, U3.2, U4.12, U4.18, U4.63; no longer U1.1, U4.P$12, U4.P$18, U4.P$63
- net I2S_BCLK: now also U4.34; no longer U4.P$34
- net I2S_DOUT: now also U4.36; no longer U4.P$36
- net I2S_LRCK: now also U4.33; no longer U4.P$33
- net I2S_MCLK: now also U4.37; no longer U4.P$37
- net LED1: now also U4.24; no longer U4.P$24
- net LOUTL: now also R9.1; no longer SJ1.1
- net MUTE: now also U4.8; no longer U4.P$8
- net N$10: now also S1.1; no longer JP1.3
- net N$12: now also U4.28; no longer U4.P$28
- net N$3: now also U4.1; no longer U4.P$1
- net N$4: now also U4.31; no longer U4.P$31
- net N$5: now also U4.5; no longer U4.P$5
- net N$6: now also U4.6; no longer U4.P$6
- net N$7: now also S1.3; no longer JP1.1
- net N$8: now also U4.47; no longer U4.P$47
- net NRST: now also U4.7; no longer U4.P$7
- net PLAYOUT: now also U4.25; no longer U4.P$25
- net RXD: now also U4.43; no longer U4.P$43
- net SD_CD: now also U4.26; no longer U4.P$26
- net SD_CK: now also U4.53; no longer U4.P$53
- net SD_CMD: now also U4.54; no longer U4.P$54
- net SD_D0: now also U4.39; no longer U4.P$39
- net SD_D1: now also U4.40; no longer U4.P$40
- net SD_D2: now also U4.51; no longer U4.P$51
- net SD_D3: now also U4.52; no longer U4.P$52
- net TRIG00: now also S2.3, U4.14; no longer U4.P$14
- net TRIG01: now also U4.15; no longer U4.P$15
- net TRIG02: now also U4.16; no longer U4.P$16
- net TRIG03: now also U4.17; no longer U4.P$17
- net TRIG04: now also U4.20; no longer U4.P$20
- net TRIG05: now also U4.21; no longer U4.P$21
- net TRIG06: now also U4.22; no longer U4.P$22
- net TRIG07: now also U4.23; no longer U4.P$23
- net TRIG08: now also U4.61; no longer U4.P$61
- net TRIG09: now also U4.62; no longer U4.P$62
- net TRIG10: now also U4.29; no longer U4.P$29
- net TRIG11: now also U4.44; no longer U4.P$44
- net TRIG12: now also U4.45; no longer U4.P$45
- net TRIG13: now also U4.46; no longer U4.P$46
- net TRIG14: now also U4.49; no longer U4.P$49
- net TRIG15: now also U4.50; no longer U4.P$50
- net TXD: now also U4.42; no longer U4.P$42
- net VCC: now also U4.13, U4.19, U4.32, U4.48, U4.64; no longer U4.P$13, U4.P$19, U4.P$32, U4.P$48, U4.P$64
- net VIN_9V: now also U3.1, U3.3; no longer U1.3
Routing:
- net N$35: track 7.30 -> 35.0 mm
- net AMPIN: track 25.9 -> 0.00 mm, vias 2 -> 0
- net N$10: track 8.04 -> 31.0 mm, vias 0 -> 2
- net BOOT0: track 42.3 -> 54.4 mm
- net +5V: track 90.0 -> 82.4 mm
- net VCC: track 317.6 -> 323.7 mm
- net MUTE: track 26.6 -> 32.5 mm
- net N$7: track 14.2 -> 8.36 mm
- net VIN_9V: track 24.1 -> 27.3 mm
- net GND: track 36.7 -> 34.8 mm, vias 20 -> 21
- net TRIG00: track 40.1 -> 41.9 mm
- net LOUTL: track 17.5 -> 19.4 mm, vias 0 -> 2
- net PLAYOUT: track 31.3 -> 32.4 mm
Other:
- board text added: "BOOT0"
- board text added: "LOAD"
- board text added: "RUN"
- board text added: "WAV Trigger"
- board text added: "v04"
- board text removed: "AMPIN"
- board text removed: "BT0"
- board text removed: "MP3 Trigger Pro"
- board text removed: "v30"

Commit message: Next round of protos ready for order, v04
Parts:
- removed U3: MIC5219 5V, SparkFun-PowerIC:SOT23-5
- added R49: 240, SparkFun-Resistors:0603-RES
- added R50: 715, SparkFun-Resistors:0603-RES
- added U1: (no value), SparkFun-PowerIC:SOT223
- R25, R26, R27, R28, R29, R30, R31, R32, R41, R42, R43, R44, R45, R46, R47, R48: value 10K -> DNP
- moved C1 10.1 mm to (16.5, 40.6), turned to 270 degrees
- moved C3 2.54 mm to (22.9, 55.9), turned to 90 degrees
- moved S1 1.40 mm to (10.5, 55.4)
- moved R16 1.27 mm to (17.8, 55.9), turned to 90 degrees
- moved J1 1.27 mm to (3.81, 44.5)
- moved C31 1.14 mm to (61.0, 52.1)
Connections:
- new net BUTTON: S2.3, U4.27
- new net N$13: R49.2, R50.2, U1.1
- net +5V: now also R49.1, U1.2, U1.4; no longer U3.5
- net GND: now also R50.1; no longer J3.CD2, U3.2
- net SD_CD: now also J3.CD2
- net TRIG00: no longer S2.3
- net VIN_9V: now also U1.3; no longer U3.1, U3.3
Routing:
- net BUTTON: track 0.00 -> 47.2 mm, vias 0 -> 4
- net TRIG00: track 41.9 -> 16.7 mm
- net +5V: track 82.4 -> 94.9 mm
- net N$13: track 0.00 -> 7.82 mm
- net VIN_9V: track 27.3 -> 23.9 mm
- net N$7: track 8.36 -> 6.57 mm
- net SD_CD: track 41.8 -> 43.5 mm, vias 4 -> 5
- net N$10: track 31.0 -> 29.6 mm
- net BOOT0: track 54.4 -> 53.6 mm
- net TRIG11: track 18.7 -> 19.4 mm
- net GND: vias 21 -> 24
Other:
- board text added: "5Vin"
- board text added: "BLK"
- board text added: "GRN"
- board text added: "SPKR"
- board text added: "T16"
- board text removed: "BOOT0"
- board text removed: "T0"

Commit message: v10 red ready
Parts:
- added J9: (no value), SparkFun-Connectors:1X02
Connections:
- removed net VIN_9V: C1.1, J1.VIN0, U1.3
- new net VIN: C1.1, J1.VIN0, J9.2, U1.3
- net GND: now also J9.1
Routing:
- net VIN: track 0.00 -> 37.6 mm
- net VIN_9V: track 23.9 -> 0.00 mm
Other:
- board text added: "VIN"
- board text added: "v10"
- board text removed: "v04"
Changed lines of the file:
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@@
 <wire x1="63.5" y1="58.42" x2="0" y2="58.41" width="0.2032" layer="20"/>
 <wire x1="0" y1="58.41" x2="0" y2="0" width="0.2032" layer="20"/>
-<text x="3.937" y="5.588" size="1.27" layer="16" font="vector" ratio="18" rot="MR0">v04</text>
+<text x="3.937" y="5.588" size="1.27" layer="16" font="vector" ratio="18" rot="MR0">v10</text>
 <text x="59.309" y="41.021" size="1.778" layer="21" font="vector" ratio="15">+</text>
 <text x="59.309" y="38.481" size="1.778" layer="21" font="vector" ratio="15">-</text>
@@
 <text x="63.119" y="22.733" size="0.8128" layer="21" font="vector" ratio="15" rot="R180">BLK</text>
 <text x="63.119" y="6.096" size="0.8128" layer="21" font="vector" ratio="15" rot="R180">GRN</text>
+<text x="2.794" y="32.512" size="1.016" layer="21" font="vector" ratio="15">GND</text>
+<text x="2.794" y="35.052" size="1.016" layer="21" font="vector" ratio="15">VIN</text>
 </plain>
 <attributes>
@@
 <element name="R50" library="SparkFun-Resistors" package="0603-RES" value="715" x="20.32" y="55.88" rot="R270"/>
 <element name="U1" library="SparkFun-PowerIC" package="SOT223" value="" x="18.034" y="48.26" rot="R180"/>
+<element name="J9" library="SparkFun-Connectors" package="1X02" value="" x="1.27" y="33.02" rot="R90"/>
 </elements>
 <signals>
-<signal name="VIN_9V">
-<contactref element="J1" pad="VIN0"/>
-<contactref element="C1" pad="1"/>
-<contactref element="U1" pad="3"/>
-<wire x1="3.81" y1="50.15" x2="3.81" y2="48.514" width="0.254" layer="1"/>
-<wire x1="3.81" y1="48.514" x2="4.318" y2="48.006" width="0.254" layer="1"/>
-<wire x1="4.318" y1="48.006" x2="14.478" y2="48.006" width="0.254" layer="1"/>
-<wire x1="14.478" y1="48.006" x2="15.748" y2="49.276" width="0.254" layer="1"/>
-<wire x1="15.748" y1="49.276" x2="15.748" y2="51.3334" width="0.254" layer="1"/>
-<wire x1="15.748" y1="51.3334" x2="15.7226" y2="51.3588" width="0.254" layer="1"/>
-<wire x1="14.478" y1="42.799" x2="14.478" y2="48.006" width="0.254" layer="1"/>
-<wire x1="14.478" y1="42.799" x2="14.986" y2="42.291" width="0.254" layer="1"/>
-<wire x1="14.986" y1="42.291" x2="16.459" y2="42.291" width="0.254" layer="1"/>
-<wire x1="16.459" y1="42.291" x2="16.51" y2="42.24" width="0.254" layer="1"/>
-</signal>
 <signal name="GND">
 <contactref element="C2" pad="2"/>
@@
 <via x="25.4" y="55.88" extent="1-16" drill="0.254"/>
 <via x="36.83" y="56.896" extent="1-16" drill="0.254"/>
+<contactref element="J9" pad="1"/>
 </signal>
 <signal name="+5V">
@@
 <wire x1="4.064" y1="24.765" x2="2.667" y2="24.765" width="0.254" layer="1"/>
 <wire x1="2.667" y1="24.765" x2="1.397" y2="26.035" width="0.254" layer="1"/>
-<wire x1="1.397" y1="26.035" x2="1.397" y2="31.242" width="0.254" layer="1"/>
-<wire x1="1.397" y1="31.242" x2="3.048" y2="32.893" width="0.254" layer="1"/>
-<wire x1="3.048" y1="32.893" x2="8.763" y2="32.893" width="0.254" layer="1"/>
+<wire x1="1.397" y1="26.035" x2="1.397" y2="30.988" width="0.254" layer="1"/>
+<wire x1="5.588" y1="32.893" x2="8.763" y2="32.893" width="0.254" layer="1"/>
 <wire x1="8.763" y1="32.893" x2="10.287" y2="34.417" width="0.254" layer="1"/>
 <wire x1="10.287" y1="34.417" x2="18.415" y2="34.417" width="0.254" layer="1"/>
@@
 <wire x1="39.878" y1="25.908" x2="39.43" y2="26.356" width="0.254" layer="1"/>
 <wire x1="39.43" y1="26.356" x2="39.43" y2="27.34" width="0.254" layer="1"/>
+<wire x1="1.397" y1="30.988" x2="1.778" y2="31.369" width="0.254" layer="1"/>
+<wire x1="1.778" y1="31.369" x2="4.064" y2="31.369" width="0.254" layer="1"/>
+<wire x1="4.064" y1="31.369" x2="5.588" y2="32.893" width="0.254" layer="1"/>
 </signal>
 <signal name="N$3">
@@
 <wire x1="4.953" y1="6.604" x2="4.953" y2="7.747" width="0.254" layer="1"/>
 </signal>
+<signal name="VIN">
+<contactref element="J1" pad="VIN0"/>
+<contactref element="C1" pad="1"/>
+<contactref element="U1" pad="3"/>
+<wire x1="3.81" y1="50.15" x2="3.81" y2="48.514" width="0.254" layer="1"/>
+<wire x1="3.81" y1="48.514" x2="4.318" y2="48.006" width="0.254" layer="1"/>
+<wire x1="4.318" y1="48.006" x2="14.478" y2="48.006" width="0.254" layer="1"/>
+<wire x1="14.478" y1="48.006" x2="15.748" y2="49.276" width="0.254" layer="1"/>
+<wire x1="15.748" y1="49.276" x2="15.748" y2="51.3334" width="0.254" layer="1"/>
+<wire x1="15.748" y1="51.3334" x2="15.7226" y2="51.3588" width="0.254" layer="1"/>
+<wire x1="14.478" y1="42.799" x2="14.478" y2="48.006" width="0.254" layer="1"/>
+<wire x1="14.478" y1="42.799" x2="14.986" y2="42.291" width="0.254" layer="1"/>
+<wire x1="14.986" y1="42.291" x2="16.459" y2="42.291" width="0.254" layer="1"/>
+<wire x1="16.459" y1="42.291" x2="16.51" y2="42.24" width="0.254" layer="1"/>
+<contactref element="J9" pad="2"/>
+<wire x1="1.27" y1="35.56" x2="1.27" y2="44.958" width="0.254" layer="1"/>
+<wire x1="1.27" y1="44.958" x2="4.318" y2="48.006" width="0.254" layer="1"/>
+</signal>
 </signals>

Commit message: v10, frame update
Parts:
- removed CC_TEXT1: CREATIVE_COMMONS, SparkFun-Aesthetics:CREATIVE_COMMONS
- added FRAME2: FRAME-LEDGER, SparkFun-Aesthetics:CREATIVE_COMMONS
Changed lines of the file:
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@@
 <text x="25.146" y="35.687" size="1.778" layer="21" font="vector" ratio="15">WAV Trigger</text>
 <text x="24.511" y="33.147" size="1.778" layer="21" font="vector" ratio="15">robertsonics</text>
-<text x="48.26" y="-11.43" size="1.778" layer="25" font="vector" ratio="15">Jamie Robertson, Jordan McConnell</text>
+<text x="17.78" y="-24.13" size="1.778" layer="25" font="vector" ratio="15">Jamie Robertson, Jordan McConnell</text>
 <text x="51.181" y="11.938" size="0.8128" layer="21" font="vector" ratio="15">LED</text>
 <text x="39.497" y="36.576" size="1.778" layer="22" font="vector" ratio="15" rot="MR0">WAV Trigger</text>
@@
 <element name="R31" library="SparkFun-Passives" package="0603-RES" value="DNP" x="36.703" y="8.89" rot="R90"/>
 <element name="R32" library="SparkFun-Passives" package="0603-RES" value="DNP" x="33.401" y="8.89" rot="R90"/>
-<element name="CC_TEXT1" library="SparkFun-Aesthetics" package="CREATIVE_COMMONS" value="CREATIVE_COMMONS" x="17.78" y="-10.16"/>
 <element name="LOGO1" library="SparkFun-Aesthetics" package="OSHW-LOGO-L" value="OSHW-LOGOL" x="31.75" y="3.302" rot="MR0"/>
 <element name="LOGO2" library="SparkFun-Aesthetics" package="SFE-NEW-WEBLOGO" value="LOGO-SFENEW" x="40.64" y="30.48" rot="MR0"/>
@@
 <element name="U1" library="SparkFun-PowerIC" package="SOT223" value="" x="18.034" y="48.26" rot="R180"/>
 <element name="J9" library="SparkFun-Connectors" package="1X02" value="" x="1.27" y="33.02" rot="R90"/>
+<element name="FRAME2" library="SparkFun-Aesthetics" package="CREATIVE_COMMONS" value="FRAME-LEDGER" x="17.78" y="-20.32"/>
 </elements>
 <signals>

Commit message: Added local micro fiducials
Parts:
- added FID1, FID2: FIDUCIALUFIDUCIAL, SparkFun-Aesthetics:MICRO-FIDUCIAL

Commit message: updated v10, changed C24-25 values to improve audio quality
Parts:
- C24, C25: value 0.1uF -> 2.2uF

Commit message: changed micro fid to regular
also deleted "wrong" panel, re-doing it
Parts:
- FID1, FID2: value FIDUCIALUFIDUCIAL -> FIDUCIAL1X2; device SparkFun-Aesthetics:MICRO-FIDUCIAL -> SparkFun-Aesthetics:FIDUCIAL-1X2
- moved FID1 4.06 mm to (5.08, 52.8)
- moved FID2 0.51 mm to (58.4, 5.84)
