File: Production Files/wavtrigger-Panel-v11.brd (EAGLE design)
At the start: 147.8 x 139.7 mm, 439 parts, among them J1 5.5x2.1mm Barrel, J10 5.5x2.1mm Barrel, J12 USD-SOCKETNEW, J15 M08X2, J17 M08X2, J19 5.5x2.1mm Barrel, J21 USD-SOCKETNEW, J24 M08X2, J26 M08X2, J28 5.5x2.1mm Barrel, J3 USD-SOCKETNEW, J30 USD-SOCKETNEW, J33 M08X2, J35 M08X2, J6 M08X2, J7 M08X2, U11 STM32F405RG, U12 MIC5323-3.3, U13 PCM5100, U14 LM4990, U16 STM32F405RG, U17 MIC5323-3.3, U18 PCM5100, U19 LM4990, U2 MIC5323-3.3, U3 STM32F405RG, U4 STM32F405RG, U5 PCM5100, U6 LM4990, U7 MIC5323-3.3, U8 PCM5100, U9 LM4990, Y1 8MHz, Y2 8MHz, Y3 8MHz, Y4 8MHz

Commit message: created panel v11
deleted panel v10
Parts:
- removed E$4: (no value), SparkFun-Aesthetics:FIDUCIAL-1X2
- added C113: 2200pF, SparkFun-Capacitors:0603-CAP
- added C114, C115: 1uF, SparkFun-Capacitors:0603-CAP
- added C116: .39uF, SparkFun-Capacitors:0603-CAP
- added E$6: (no value), SparkFun-Aesthetics:FIDUCIAL-1X2
- added J37, J40: (no value), SparkFun-Connectors:1X04
- added J38: M08X2, SparkFun-Connectors:2X8
- added J39: M02PTH, SparkFun-Connectors:1X02
- added TP1, TP2, TP3, TP4: TEST-POINTTP_15TH_THRU, SparkFun-Passives:TP_15TH
- C100, C43, C71, C72: value 0.1uF -> 33pF
- C101: value 2.2uF -> 33pF
- C104, C24, C25, C46, C50, C51, C68, C75, C79: value 0.1uF -> 2.2uF
- C108, C80: value 10uF -> 2.2uF
- C109: value 2200pF -> 2.2uF
- C110, C81: value 2200pF -> 0.1uF
- C111: value 1uF -> 10uF
- C112, C55, C83, C84: value 1uF -> 2200pF
- C32: value 2.2uF -> 0.1uF; device SparkFun-Capacitors:0805 -> SparkFun-Capacitors:0603-CAP
- C33, C89: value 10uF -> 2.2uF; device SparkFun-Capacitors:1210 -> SparkFun-Capacitors:0805
- C34, C92: value 0.1uF -> 10uF; device SparkFun-Capacitors:0603-CAP -> SparkFun-Capacitors:1210
- C35: value 1uF -> 0.1uF
- C36, C65: value 0.1uF -> 1uF
- C38, C45, C66, C73: value 2.2uF -> 0.1uF
- C39: value 4.7uF -> 2.2uF
- C40: value 0.1uF -> 4.7uF
- C41, C70: value 33pF -> 0.1uF
- C52: value 10uF -> 0.1uF
- C53, C82: value 2200pF -> 10uF
- C57, C85: value 10uF -> 1uF; device SparkFun-Capacitors:0805 -> SparkFun-Capacitors:0603-CAP
- C58: value 2.2uF -> .39uF; device SparkFun-Capacitors:0805 -> SparkFun-Capacitors:0603-CAP
- C59: value 0.1uF -> 10uF; device SparkFun-Capacitors:0603-CAP -> SparkFun-Capacitors:0805
- C6: value 10uF -> .39uF; device SparkFun-Capacitors:0805 -> SparkFun-Capacitors:0603-CAP
- C61: value 10uF -> 0.1uF; device SparkFun-Capacitors:1210 -> SparkFun-Capacitors:0603-CAP
- C62, C8: value 0.1uF -> 2.2uF; device SparkFun-Capacitors:0603-CAP -> SparkFun-Capacitors:0805
- C63: value 1uF -> 10uF; device SparkFun-Capacitors:0603-CAP -> SparkFun-Capacitors:1210
- C67, C95: value 4.7uF -> 0.1uF
- C69, C98: value 33pF -> 4.7uF
- C7, C88: value 2.2uF -> 10uF
- C86: value 2.2uF -> 1uF; device SparkFun-Capacitors:0805 -> SparkFun-Capacitors:0603-CAP
- C87: value 0.1uF -> .39uF
- C91: value 1uF -> 2.2uF; device SparkFun-Capacitors:0603-CAP -> SparkFun-Capacitors:0805
- C94: value 2.2uF -> 1uF
- C97: value 33pF -> 2.2uF
- E$1: device SparkFun-Aesthetics:FIDUCIAL-1.5X3 -> SparkFun-Retired:FIDUCIAL-1.5X3
- FID1, FID2, FID3, FID4, FID5, FID6, FID7, FID8: value FIDUCIALUFIDUCIAL -> FIDUCIAL1X2; device SparkFun-Aesthetics:MICRO-FIDUCIAL -> SparkFun-Aesthetics:FIDUCIAL-1X2
- J1: device SparkFun-Connectors:POWER_JACK_SMD -> Testing:POWER_JACK_SMD_OVERPASTE_REDBOARD_0603
- J10: value 5.5x2.1mm Barrel -> (none); device SparkFun-Connectors:POWER_JACK_SMD -> SparkFun-Connectors:1X04
- J11: value (none) -> 5.5x2.1mm Barrel; device SparkFun-Connectors:AUDIO-JACK-3.5MM-SMD -> Testing:POWER_JACK_SMD_OVERPASTE_REDBOARD_0603
- J12: value USD-SOCKETNEW -> (none); device robertsonics:MICRO-SD-SOCKET-PP -> SparkFun-Connectors:AUDIO-JACK-3.5MM-SMD
- J13: value (none) -> USD-SOCKETNEW; device SparkFun-Connectors:1X02 -> robertsonics:MICRO-SD-SOCKET-PP
- J14: value (none) -> M02PTH; device SparkFun-Connectors:1X06 -> SparkFun-Connectors:1X02
- J15, J35: value M08X2 -> (none); device SparkFun-Connectors:2X8 -> SparkFun-Connectors:1X06
- J16: value (none) -> M08X2; device SparkFun-Connectors:1X04 -> SparkFun-Connectors:2X8
- J17: value M08X2 -> (none); device SparkFun-Connectors:2X8 -> SparkFun-Connectors:1X04
- J18, J36: value (none) -> M08X2; device SparkFun-Connectors:1X02 -> SparkFun-Connectors:2X8
- J19: value 5.5x2.1mm Barrel -> M02PTH; device SparkFun-Connectors:POWER_JACK_SMD -> SparkFun-Connectors:1X02
- J20: device SparkFun-Connectors:AUDIO-JACK-3.5MM-SMD -> SparkFun-Connectors:1X04
- J21: value USD-SOCKETNEW -> 5.5x2.1mm Barrel; device robertsonics:MICRO-SD-SOCKET-PP -> Testing:POWER_JACK_SMD_OVERPASTE_REDBOARD_0603
- J22: device SparkFun-Connectors:1X02 -> SparkFun-Connectors:AUDIO-JACK-3.5MM-SMD
- J23: value (none) -> USD-SOCKETNEW; device SparkFun-Connectors:1X06 -> robertsonics:MICRO-SD-SOCKET-PP
- J24: value M08X2 -> M02PTH; device SparkFun-Connectors:2X8 -> SparkFun-Connectors:1X02
- J25: device SparkFun-Connectors:1X04 -> SparkFun-Connectors:1X06
- J27: device SparkFun-Connectors:1X02 -> SparkFun-Connectors:1X04
- J28: value 5.5x2.1mm Barrel -> M08X2; device SparkFun-Connectors:POWER_JACK_SMD -> SparkFun-Connectors:2X8
- J29: value (none) -> M02PTH; device SparkFun-Connectors:AUDIO-JACK-3.5MM-SMD -> SparkFun-Connectors:1X02
- J30: value USD-SOCKETNEW -> (none); device robertsonics:MICRO-SD-SOCKET-PP -> SparkFun-Connectors:1X04
- J31: value (none) -> 5.5x2.1mm Barrel; device SparkFun-Connectors:1X02 -> Testing:POWER_JACK_SMD_OVERPASTE_REDBOARD_0603
- J32: device SparkFun-Connectors:1X06 -> SparkFun-Connectors:AUDIO-JACK-3.5MM-SMD
- J33: value M08X2 -> USD-SOCKETNEW; device SparkFun-Connectors:2X8 -> robertsonics:MICRO-SD-SOCKET-PP
- J34: value (none) -> M02PTH; device SparkFun-Connectors:1X04 -> SparkFun-Connectors:1X02
- J5, J9: value (none) -> M02PTH
- LOGO12, LOGO6, LOGO9: value LOGO-SFESK -> SFE_LOGO_FLAME.2_INCH; device SparkFun-Aesthetics:SFE-LOGO-FLAME -> SparkFun-Aesthetics:SFE_LOGO_FLAME_.2
- LOGO3: value LOGO-SFESK -> OSHW-LOGOL; device SparkFun-Aesthetics:SFE-LOGO-FLAME -> SparkFun-Aesthetics:OSHW-LOGO-L
- LOGO4: value OSHW-LOGOL -> SFE_LOGO_FLAME.2_INCH; device SparkFun-Aesthetics:OSHW-LOGO-L -> SparkFun-Aesthetics:SFE_LOGO_FLAME_.2
- moved C58 123.5 mm to (127.8, 46.7)
- moved J20 121.0 mm to (137.2, 32.3), turned to 90 degrees
- moved J29 120.5 mm to (11.4, 103.1), turned to 90 degrees
- moved C57 118.6 mm to (138.4, 58.9), turned to 180 degrees
- moved E$5 114.0 mm to (143.1, 9.40), turned to 0 degrees
- moved J19 98.9 mm to (78.7, 39.9), turned to 90 degrees
- moved J24 65.5 mm to (72.4, 109.5), turned to 90 degrees
- moved J27 61.4 mm to (72.4, 95.5)
- moved LOGO3 59.5 mm to (109.2, 10.2), flipped to the bottom
- moved LOGO4 59.5 mm to (57.4, 39.4), flipped to the top
- moved J31 58.6 mm to (81.3, 114.6), turned to 0 degrees
- moved J16 58.5 mm to (86.4, 8.13), turned to 0 degrees
- moved J15 56.6 mm to (139.7, 27.2), turned to 270 degrees
- moved J28 55.1 mm to (47.0, 71.4)
- moved J11 49.9 mm to (81.3, 51.3), turned to 0 degrees
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Connections:
- removed net N$115 (its old number): C97.2, U16.5, Y4.2
- removed net N$131 (its old number): J32.3, SJ13.1
- removed net N$133 (its old number): J33.4, R168.1, R181.1
- removed net N$134 (its old number): J33.6, R169.1, R180.1
- removed net N$135 (its old number): J33.8, R170.1, R179.1
- removed net N$136 (its old number): J33.10, R171.1, R178.1
- removed net N$50 (its old number): C55.2, U9.2, U9.3
- removed net N$57 (its old number): J14.3, SJ1.1
- removed net N$58 (its old number): J15.2, R67.1, R82.1
- removed net N$76 (its old number): C62.2, U11.1
- removed net N$89 (its old number): J23.4, R112.2
- removed net N$94 (its old number): J23.3, SJ9.1
- removed net N$95 (its old number): J24.2, R117.1, R132.1
- removed net N$96 (its old number): J24.4, R118.1, R131.1
- removed net N$97 (its old number): J24.6, R119.1, R130.1
- new net I2S_DI: J10.2, U4.35
- new net I2S_DI1: J20.2, U3.35
- new net I2S_DI2: J30.2, U11.35
- new net I2S_DI3: J40.2, U16.35
- new net N$111: J28.10, R137.1, R144.1
- new net N$122: C101.2, U16.6, Y4.1
- new net N$123: C104.1, U16.47
- new net N$125: C108.2, U18.2
- new net N$127: C109.1, U18.5
- new net N$130: C114.2, U19.2, U19.3
- new net N$148: J38.6, R185.1, R196.1
- new net N$149: J38.8, R186.1, R195.1
- new net N$150: J38.10, R187.1, R194.1
- new net N$151: J38.12, R188.1, R193.1
- new net N$152: J38.14, R189.1, R192.1
- new net N$153: J38.16, R190.1, R191.1
- new net N$155: C116.1, R159.1
- new net N$156: TP4.P$1, U16.4
- new net N$48: C50.1, U8.4
- new net N$49: C51.1, U8.5
- new net N$54: J15.4, R62.2
- new net N$74: J18.14, R89.1, R92.1
- new net N$85: C78.2, U13.18
- new net N$86: C79.2, U13.2
- new net N$88: C80.1, U13.5
- new net N$91: C85.2, U14.2, U14.3
- new net N$93: J25.4, R112.2
- net +5V1: now also C57.2, C8.1, J17.4; no longer C56.2, C6.1, J16.4
- net +5V2: now also C59.1, C60.1, C86.2, J27.4; no longer C57.1, C58.1, C84.2, J25.4
- net +5V3: now also C115.2, C88.1, C89.1, J37.4; no longer C112.2, C85.1, C86.1, J34.4
- net GND1: now also C34.2, C41.2, C43.1, C46.2, C47.1, C48.2, C49.1, C51.2, C57.1, J11.GND, J11.P$4, J12.SLEEVE, J13.6, J13.GND1, J13.GND3, J16.11, J16.13, J16.15, J16.3, J16.5, J16.7, J16.9, J18.11, J18.13, J18.15, J18.3, J18.5, J18.7, J18.9, J19.1; no longer C35.2, C41.1, C43.2, C46.1, C47.2, C48.1, C50.2, C51.1, C6.2, J10.GND, J10.P$4, J11.SLEEVE, J12.6, J12.GND1, J12.GND3, J14.1, J15.11, J15.13, J15.15, J15.3, J15.5, J15.7, J15.9, J17.11, J17.13, J17.15, J17.3, J17.5, J17.7, J17.9
- net GND2: now also C62.2, C69.2, C70.2, C71.1, C72.1, C74.2, C77.2, C78.1, C80.2, C85.1, C86.1, J21.GND, J21.P$4, J22.SLEEVE, J23.6, J23.GND1, J23.GND3, J28.1, J28.11, J28.13, J28.15, J28.3, J28.5, J28.7, J28.9, J29.1; no longer C57.2, C58.2, C64.2, C69.1, C70.1, C71.2, C72.2, C74.1, C78.2, C79.1, C80.1, J19.GND, J19.P$4, J20.SLEEVE, J21.6, J21.GND1, J21.GND3, J23.1, J24.1, J24.11, J24.13, J24.15, J24.3, J24.5, J24.7, J24.9
- net GND3: now also C100.1, C101.1, C102.2, C104.2, C105.1, C109.2, C113.1, C114.1, C115.1, C90.2, C97.2, C98.2, J31.GND, J31.P$4, J32.SLEEVE, J33.6, J33.GND1, J33.GND3, J36.11, J36.13, J36.15, J36.3, J36.5, J36.7, J36.9, J37.1, J38.1, J38.11, J38.13, J38.15, J38.3, J38.5, J38.7, J38.9, J39.1; no longer C100.2, C101.2, C102.1, C104.1, C108.1, C109.1, C85.2, C86.2, C87.2, C93.2, C97.1, C98.1, J28.GND, J28.P$4, J29.SLEEVE, J30.6, J30.GND1, J30.GND3, J32.1, J33.1, J33.11, J33.13, J33.15, J33.3, J33.5, J33.7, J33.9, J34.1, J35.11, J35.13, J35.15, J35.3, J35.5, J35.7, J35.9
- net I2S_BCLK: now also J10.3
- net I2S_BCLK1: now also J20.3
- net I2S_BCLK2: now also J30.3
- net I2S_BCLK3: now also J40.3
- net I2S_LRCK: now also J10.4
- net I2S_LRCK1: now also J20.4
- net I2S_LRCK2: now also J30.4
- net I2S_LRCK3: now also J40.4
- net I2S_MCLK: now also J10.1
- net I2S_MCLK1: now also J20.1
- net I2S_MCLK2: now also J30.1
- net I2S_MCLK3: now also J40.1
- net LOUTL: now also C6.2; no longer R9.1
- net LOUTL1: now also C54.2, C58.2, J12.TIP; no longer C53.2, J11.TIP, R59.1
- net LOUTL2: now also C83.2, C87.2, J22.TIP; no longer C81.2, J20.TIP, R109.1
- net LOUTL3: now also C112.2, C116.2, J32.TIP; no longer C109.2, J29.TIP, R159.1
- net LOUTR1: now also C55.2, J12.RING; no longer C54.2, J11.RING
- net LOUTR2: now also C84.2, J22.RING; no longer C82.2, J20.RING
- net LOUTR3: now also C113.2, J32.RING; no longer C110.2, J29.RING
- net N$100: now also J26.4, R118.1, R131.1; no longer J24.12, R122.1, R127.1
- net N$101: now also J26.6, R119.1, R130.1; no longer J24.14, R123.1, R126.1
- net N$102: now also J26.8, R120.1, R129.1; no longer J24.16, R124.1, R125.1
- net N$103: now also J26.10, R121.1, R128.1; no longer J26.2, R133.1, R148.1
- net N$104: now also J26.12, R122.1, R127.1; no longer J26.4, R134.1, R147.1
- net N$105: now also J26.14, R123.1, R126.1; no longer J26.6, R135.1, R146.1
- net N$106: now also J26.16, R124.1, R125.1; no longer J26.8, R136.1, R145.1
- net N$107: now also J28.2, R133.1, R148.1; no longer J26.10, R137.1, R144.1
- net N$108: now also J28.4, R134.1, R147.1; no longer J26.12, R138.1, R143.1
- net N$109: now also J28.6, R135.1, R146.1; no longer J26.14, R139.1, R142.1
- net N$110: now also J28.8, R136.1, R145.1; no longer J26.16, R140.1, R141.1
- net N$112: now also J28.12, R138.1, R143.1; no longer C87.1, U17.4
- net N$113: now also J28.14, R139.1, R142.1; no longer C90.2, U16.1
- net N$114: now also J28.16, R140.1, R141.1; no longer C94.1, U16.31
- net N$116: now also C87.1, R109.1; no longer C98.2, U16.6, Y4.1
- net N$117: now also TP3.P$1, U11.4; no longer C101.1, U16.47
- net N$118: now also C90.1, U17.4; no longer C104.2, U18.18
- net N$119: now also C93.2, U16.1; no longer C105.2, U18.2
- net N$120: now also C97.1, U16.31; no longer C105.1, U18.4
- net N$121: now also C100.2, U16.5, Y4.2; no longer C106.1, U18.5
- net N$124: now also C107.2, U18.18; no longer C111.2, U19.2, U19.3
- net N$126: now also C108.1, U18.4; no longer J32.4, R162.2
- net N$132: now also J35.4, R162.2; no longer J33.2, R167.1, R182.1
- net N$137: now also J35.3, SJ13.1; no longer J33.12, R172.1, R177.1
- net N$138: now also J36.2, R167.1, R182.1; no longer J33.14, R173.1, R176.1
- net N$139: now also J36.4, R168.1, R181.1; no longer J33.16, R174.1, R175.1
- net N$140: now also J36.6, R169.1, R180.1; no longer J35.2, R183.1, R198.1
- net N$141: now also J36.8, R170.1, R179.1; no longer J35.4, R184.1, R197.1
- net N$142: now also J36.10, R171.1, R178.1; no longer J35.6, R185.1, R196.1
- net N$143: now also J36.12, R172.1, R177.1; no longer J35.8, R186.1, R195.1
- net N$144: now also J36.14, R173.1, R176.1; no longer J35.10, R187.1, R194.1
- net N$145: now also J36.16, R174.1, R175.1; no longer J35.12, R188.1, R193.1
- net N$146: now also J38.2, R183.1, R198.1; no longer J35.14, R189.1, R192.1
- net N$147: now also J38.4, R184.1, R197.1; no longer J35.16, R190.1, R191.1
- net N$21: now also C6.1, R9.1; no longer C8.1, U7.4
- net N$22: now also TP1.P$1, U4.4; no longer C34.2, U3.1
- net N$31: now also C32.1, U7.4; no longer C38.1, U3.31
- net N$33: now also C35.2, U3.1; no longer C41.2, U3.5, Y2.2
- net N$34: now also C39.1, U3.31; no longer C42.2, U3.6, Y2.1
- net N$43: now also C42.2, U3.5, Y2.2; no longer C45.1, U3.47
- net N$44: now also C43.2, U3.6, Y2.1; no longer C48.2, U8.18
- net N$45: now also C46.1, U3.47; no longer C49.2, U8.2
- net N$46: now also C49.2, U8.18; no longer C49.1, U8.4
- net N$47: now also C50.2, U8.2; no longer C50.1, U8.5
- net N$52: now also C56.2, U9.2, U9.3; no longer J14.4, R62.2
- net N$59: now also J15.3, SJ1.1; no longer J15.4, R68.1, R81.1
- net N$60: now also J16.2, R67.1, R82.1; no longer J15.6, R69.1, R80.1
- net N$61: now also J16.4, R68.1, R81.1; no longer J15.8, R70.1, R79.1
- net N$62: now also J16.6, R69.1, R80.1; no longer J15.10, R71.1, R78.1
- net N$63: now also J16.8, R70.1, R79.1; no longer J15.12, R72.1, R77.1
- net N$64: now also J16.10, R71.1, R78.1; no longer J15.14, R73.1, R76.1
- net N$65: now also J16.12, R72.1, R77.1; no longer J15.16, R74.1, R75.1
- net N$66: now also J16.14, R73.1, R76.1; no longer J17.2, R83.1, R98.1
- net N$67: now also J16.16, R74.1, R75.1; no longer J17.4, R84.1, R97.1
- net N$68: now also J18.2, R83.1, R98.1; no longer J17.6, R85.1, R96.1
- net N$69: now also J18.4, R84.1, R97.1; no longer J17.8, R86.1, R95.1
- net N$70: now also J18.6, R85.1, R96.1; no longer J17.10, R87.1, R94.1
- net N$71: now also J18.8, R86.1, R95.1; no longer J17.12, R88.1, R93.1
- net N$72: now also J18.10, R87.1, R94.1; no longer J17.14, R89.1, R92.1
- net N$73: now also J18.12, R88.1, R93.1; no longer J17.16, R90.1, R91.1
- net N$75: now also J18.16, R90.1, R91.1; no longer C59.1, U12.4
- net N$77: now also C58.1, R59.1; no longer C66.1, U11.31
- net N$78: now also TP2.P$1, U3.4; no longer C69.2, U11.5, Y3.2
- net N$79: now also C61.1, U12.4; no longer C70.2, U11.6, Y3.1
- net N$80: now also C64.2, U11.1; no longer C73.1, U11.47
- net N$81: now also C68.1, U11.31; no longer C76.2, U13.18
- net N$82: now also C71.2, U11.5, Y3.2; no longer C77.2, U13.2
- net N$83: now also C72.2, U11.6, Y3.1; no longer C77.1, U13.4
- net N$84: now also C75.1, U11.47; no longer C78.1, U13.5
- net N$87: now also C79.1, U13.4; no longer C83.2, U14.2, U14.3
- net N$98: now also J25.3, SJ9.1; no longer J24.8, R120.1, R129.1
- net N$99: now also J26.2, R117.1, R132.1; no longer J24.10, R121.1, R128.1
- net PLAYOUT1: now also J17.2; no longer J16.2
- net PLAYOUT2: now also J27.2; no longer J25.2
- net PLAYOUT3: now also J37.2; no longer J34.2
- net SD_CD1: now also J13.CD1, J13.CD2; no longer J12.CD1, J12.CD2
- net SD_CD2: now also J23.CD1, J23.CD2; no longer J21.CD1, J21.CD2
- net SD_CD3: now also J33.CD1, J33.CD2; no longer J30.CD1, J30.CD2
- net SD_CK1: now also J13.5; no longer J12.5
- net SD_CK2: now also J23.5; no longer J21.5
- net SD_CK3: now also J33.5; no longer J30.5
- net SD_CMD1: now also J13.3; no longer J12.3
- net SD_CMD2: now also J23.3; no longer J21.3
- net SD_CMD3: now also J33.3; no longer J30.3
- net SD_D10: now also J23.2; no longer J21.2
- net SD_D11: now also J23.1; no longer J21.1
- net SD_D12: now also J33.8; no longer J30.8
- net SD_D13: now also J33.7; no longer J30.7
- net SD_D14: now also J33.2; no longer J30.2
- net SD_D15: now also J33.1; no longer J30.1
- net SD_D4: now also J13.8; no longer J12.8
- net SD_D5: now also J13.7; no longer J12.7
- net SD_D6: now also J13.2; no longer J12.2
- net SD_D7: now also J13.1; no longer J12.1
- net SD_D8: now also J23.8; no longer J21.8
- net SD_D9: now also J23.7; no longer J21.7
- net SPKR+1: now also J14.2; no longer J13.2
- net SPKR+2: now also J24.2; no longer J22.2
- net SPKR+3: now also J34.2; no longer J31.2
- net SPKR-1: now also J14.1; no longer J13.1
- net SPKR-2: now also J24.1; no longer J22.1
- net SPKR-3: now also J34.1; no longer J31.1
- net TXD1: now also J15.5; no longer J14.5
- net TXD2: now also J25.5; no longer J23.5
- net TXD3: now also J35.5; no longer J32.5
- net VCC1: now also C33.1, C38.1, C41.1, C45.1, C47.2, C48.1, C53.2, J13.4, J17.3; no longer C32.1, C34.1, C39.1, C43.1, C46.2, C47.1, C51.2, J12.4, J16.3
- net VCC2: now also C66.1, C69.1, C70.1, C73.1, C74.1, C76.2, C77.1, C81.2, C82.2, J23.4, J27.3; no longer C60.1, C63.1, C68.1, C71.1, C72.1, C74.2, C75.1, C79.2, C80.2, J21.4, J25.3
- net VCC3: now also C102.1, C105.2, C106.1, C110.2, C111.2, C94.1, C98.1, J33.4, J37.3; no longer C100.1, C102.2, C107.2, C108.2, C88.1, C90.1, C92.1, J30.4, J34.3
- net VIN1: now also C34.1, J11.VIN0, J19.2; no longer C33.1, J10.VIN0, J18.2
- net VIN2: now also C63.1, J21.VIN0, J29.2; no longer C61.1, J19.VIN0, J27.2
- net VIN3: now also C92.1, J31.VIN0, J39.2; no longer C89.1, J28.VIN0, J36.2
Routing:
- net N$58 (its old number): track 35.0 -> 0.00 mm
- net N$95 (its old number): track 35.0 -> 0.00 mm
- net N$99: track 5.99 -> 35.0 mm
- net N$138: track 6.04 -> 35.0 mm
- net N$60: track 6.67 -> 35.0 mm
- net N$131 (its old number): track 23.6 -> 0.00 mm
- net N$57 (its old number): track 23.6 -> 0.00 mm
- net N$94 (its old number): track 23.6 -> 0.00 mm
- net N$132: track 35.0 -> 11.5 mm
- net N$137: track 6.09 -> 26.4 mm
- net N$98: track 6.35 -> 26.4 mm
- net N$76 (its old number): track 19.9 -> 0.00 mm, vias 2 -> 0
- net N$59: track 6.99 -> 26.4 mm
- net N$22: track 19.9 -> 1.82 mm, vias 2 -> 0
- net I2S_DI1: track 0.00 -> 17.1 mm, vias 0 -> 1
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- added copper zone on layer 1, net +5V
- added copper zone on layer 16, net +5V
- added copper zone on layer 1, net +5V1
- added copper zone on layer 16, net +5V1
- added copper zone on layer 1, net +5V2
- added copper zone on layer 16, net +5V2
- added copper zone on layer 1, net +5V3
- added copper zone on layer 16, net +5V3
Other:
- outline, holes or cut-outs redrawn
- board text added: "BC"
- board text added: "DI"
- board text added: "I2S"
- board text added: "LR"
- board text added: "MC"
- board text added: "v11"
- board text removed: "v10"
